File: TankTurret/TankTurret.kicad_pcb (KiCad board)
At the start: 2 copper layers, 32 x 39.6 mm, 23 parts, among them J2 Camera, J3 SlipRing_6, P1 USB_C_Plug, U1 ESP32-WROVER-E

Commit message: camera connector
Parts:
- removed J3: SlipRing_6, Connector_JST:JST_XH_B6B-XH-A_1x06_P2.50mm_Vertical
- added C1: 100nF, Capacitor_SMD:C_0402_1005Metric, F.Cu at (123.3, 72.8)
- added C17: 1uF, Capacitor_SMD:C_0201_0603Metric, F.Cu at (125.9, 76.2)
- added C18: 100nF, Capacitor_SMD:C_0402_1005Metric, F.Cu at (123.3, 78.7)
- added C19: 1uF, Capacitor_SMD:C_0201_0603Metric, F.Cu at (125.9, 77.9)
- added C2: 1uF, Capacitor_SMD:C_0201_0603Metric, F.Cu at (125.9, 72.7)
- added C20: 100nF, Capacitor_SMD:C_0402_1005Metric, F.Cu at (123.3, 80.7)
- added C21: 1uF, Capacitor_SMD:C_0201_0603Metric, F.Cu at (125.9, 79.7)
- added C3: 4.7uF, Capacitor_SMD:C_0805_2012Metric, F.Cu at (116.0, 82.6)
- added C4: 100nF, Capacitor_SMD:C_0402_1005Metric, F.Cu at (123.3, 74.8)
- added C5: 1uF, Capacitor_SMD:C_0201_0603Metric, F.Cu at (125.9, 74.4)
- added C6: 100nF, Capacitor_SMD:C_0402_1005Metric, F.Cu at (123.3, 76.7)
- added FB1: FerriteBead, Inductor_SMD:L_0603_1608Metric, F.Cu at (123.8, 82.9)
- added J1: Conn_01x04_Socket, Connector_JST:JST_XH_B4B-XH-A_1x04_P2.50mm_Vertical, B.Cu at (81.7, 60.7)
- added R1: 4.7k, Resistor_SMD:R_0402_1005Metric, F.Cu at (120.4, 72.8)
- added R2: 4.7k, Resistor_SMD:R_0402_1005Metric, F.Cu at (120.4, 74.8)
- added R3: 10k, Resistor_SMD:R_0402_1005Metric, F.Cu at (120.4, 76.8)
- added R4: 10k, Resistor_SMD:R_0402_1005Metric, F.Cu at (120.4, 78.8)
- added R5: 33Ω, Resistor_SMD:R_0402_1005Metric, F.Cu at (120.4, 80.8)
- added U2: TLV70028_SOT353, Package_TO_SOT_SMD:SOT-23-5, F.Cu at (116.3, 74.2)
- added U4: TLV70012_SOT23-5, Package_TO_SOT_SMD:SOT-23-5, F.Cu at (116.3, 78.8)
- J2: footprint Connector_FFC-FPC:TE_2-1734839-3_1x23-1MP_P0.5mm_Horizontal -> Connector_FFC-FPC:TE_2-1734839-4_1x24-1MP_P0.5mm_Horizontal
- P1: footprint Connector_USB:USB_C_Receptacle_HCTL_HC-TYPE-C-16P-01A -> Connector_USB:USB_C_Receptacle_HRO_TYPE-C-31-M-17; moved to B.Cu
- U1: footprint PCM_Espressif:ESP32-WROVER-E -> RF_Module:ESP32-S3-WROOM-1U; moved to F.Cu
- moved C10 65.8 mm to (105.6, 75.2)
- moved C11 65.8 mm to (102.0, 90.3)
- moved C9 65.8 mm to (105.6, 72.2)
- moved R15 65.8 mm to (101.4, 71.9)
- moved R16 65.8 mm to (101.4, 74.4)
- moved C12 65.8 mm to (93.7, 95.2)
- moved C13 65.8 mm to (97.4, 76.9)
- moved C7 65.8 mm to (97.4, 71.9)
- moved C8 65.8 mm to (97.4, 74.4)
- moved L2 61.6 mm to (63.8, 89.8), turned to 90 degrees
- moved U1 59.6 mm to (65.7, 54.7)
- moved PS2 57.2 mm to (66.4, 98.5)
- moved PS1 47.1 mm to (76.5, 98.6)
- moved C14 46.3 mm to (102.6, 60.4)
- moved C15 46.3 mm to (102.6, 62.9)
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Connections:
- J2 pad 11: /GPIO34 -> /GPIO17
- J2 pad 12: /GPIO21 -> Net-(J2-XCLK)
- J2 pad 13: /GPIO35 -> /GPIO16
- J2 pad 14: unconnected-(J2-DOVDD-Pad14) -> +CAM_2V8
- J2 pad 15: unconnected-(J2-DVDD-Pad15) -> CAM_1V2
- J2 pad 16: /GPIO23 -> /GPIO7
- J2 pad 17: GND -> Net-(J2-PWDN)
- J2 pad 18: /GPIO25 -> /GPIO6
- J2 pad 20: /GPIO27 -> /GPIO5
- J2 pad 21: unconnected-(J2-AVDD-Pad21) -> Net-(J2-AVDD)
- J2 pad 22: /GPIO26 -> /GPIO4
- J2 pad 23: unconnected-(J2-AGND-Pad23) -> GND
- J2 pad 3: /GPIO18 -> /GPIO8
- J2 pad 4: /GPIO5 -> /GPIO9
- J2 pad 5: /GPIO19 -> /GPIO10
- J2 pad 6: /GPIO4 -> /GPIO11
- J2 pad 7: /GPIO36 -> /GPIO12
- J2 pad 8: /GPIO22 -> /GPIO13
- J2 pad 9: /GPIO39 -> /GPIO18
- U1 pad 1: GND -> Net-(U1-GND-Pad1)
- U1 pad 10: /GPIO25 -> unconnected-(U1-GPIO17/U1TXD/ADC2_CH6-Pad10)
- U1 pad 11: /GPIO26 -> unconnected-(U1-GPIO18/U1RXD/ADC2_CH7/CLK_OUT3-Pad11)
- U1 pad 12: /GPIO27 -> unconnected-(U1-GPIO8/TOUCH8/ADC1_CH7/SUBSPICS1-Pad12)
- U1 pad 13: /BUZZER -> unconnected-(U1-GPIO19/U1RTS/ADC2_CH8/CLK_OUT2/USB_D--Pad13)
- U1 pad 14: /IR #1 -> unconnected-(U1-GPIO20/U1CTS/ADC2_CH9/CLK_OUT1/USB_D+-Pad14)
- U1 pad 15: GND -> unconnected-(U1-GPIO3/TOUCH3/ADC1_CH2-Pad15)
- U1 pad 16: /TOP_LEDS -> unconnected-(U1-GPIO46-Pad16)
- U1 pad 17: (no net) -> unconnected-(U1-GPIO9/TOUCH9/ADC1_CH8/FSPIHD/SUBSPIHD-Pad17)
- U1 pad 18: (no net) -> unconnected-(U1-GPIO10/TOUCH10/ADC1_CH9/FSPICS0/FSPIIO4/SUBSPICS0-Pad18)
- U1 pad 19: (no net) -> unconnected-(U1-GPIO11/TOUCH11/ADC2_CH0/FSPID/FSPIIO5/SUBSPID-Pad19)
- U1 pad 20: (no net) -> unconnected-(U1-GPIO12/TOUCH12/ADC2_CH1/FSPICLK/FSPIIO6/SUBSPICLK-Pad20)
- U1 pad 21: (no net) -> unconnected-(U1-GPIO13/TOUCH13/ADC2_CH2/FSPIQ/FSPIIO7/SUBSPIQ-Pad21)
- U1 pad 22: (no net) -> unconnected-(U1-GPIO14/TOUCH14/ADC2_CH3/FSPIWP/FSPIDQS/SUBSPIWP-Pad22)
- U1 pad 24: /IR #2 -> unconnected-(U1-GPIO47/SPICLK_P/SUBSPICLK_P_DIFF-Pad24)
- U1 pad 26: /GPIO4 -> unconnected-(U1-GPIO45-Pad26)
- U1 pad 27: (no net) -> unconnected-(U1-GPIO0/BOOT-Pad27)
- U1 pad 28: (no net) -> unconnected-(U1-SPIIO6/GPIO35/FSPID/SUBSPID-Pad28)
- U1 pad 29: /GPIO5 -> unconnected-(U1-SPIIO7/GPIO36/FSPICLK/SUBSPICLK-Pad29)
- U1 pad 30: /GPIO18 -> unconnected-(U1-SPIDQS/GPIO37/FSPIQ/SUBSPIQ-Pad30)
- U1 pad 31: /GPIO19 -> unconnected-(U1-GPIO38/FSPIWP/SUBSPIWP-Pad31)
- U1 pad 32: (no net) -> unconnected-(U1-MTCK/GPIO39/CLK_OUT3/SUBSPICS1-Pad32)
- U1 pad 33: /GPIO21 -> unconnected-(U1-MTDO/GPIO40/CLK_OUT2-Pad33)
- U1 pad 34: /USB-UART RX -> unconnected-(U1-MTDI/GPIO41/CLK_OUT1-Pad34)
- U1 pad 35: /USB-UART TX -> unconnected-(U1-MTMS/GPIO42-Pad35)
- U1 pad 36: /GPIO22 -> unconnected-(U1-U0RXD/GPIO44/CLK_OUT2-Pad36)
- U1 pad 37: /GPIO23 -> unconnected-(U1-U0TXD/GPIO43/CLK_OUT1-Pad37)
- U1 pad 38: GND -> unconnected-(U1-GPIO2/TOUCH2/ADC1_CH1-Pad38)
- U1 pad 39: GND -> /BUZZER
- U1 pad 4: /GPIO36 -> unconnected-(U1-GPIO4/TOUCH4/ADC1_CH3-Pad4)
- U1 pad 5: /GPIO39 -> unconnected-(U1-GPIO5/TOUCH5/ADC1_CH4-Pad5)
- U1 pad 6: /GPIO34 -> unconnected-(U1-GPIO6/TOUCH6/ADC1_CH5-Pad6)
- U1 pad 7: /GPIO35 -> unconnected-(U1-GPIO7/TOUCH7/ADC1_CH6-Pad7)
- U1 pad 8: /I2C SCL -> unconnected-(U1-GPIO15/U0RTS/ADC2_CH4/XTAL_32K_P-Pad8)
- U1 pad 9: /I2C SDA -> unconnected-(U1-GPIO16/U0CTS/ADC2_CH5/XTAL_32K_N-Pad9)
Routing:
- added copper zone on B.Cu, net GND
Other:
- board size 32 x 39.6 mm -> 35 x 60 mm

Commit message: bits
Parts:
- removed C15: 100nF, Capacitor_SMD:C_0603_1608Metric
- removed C16: 18pF, Capacitor_SMD:C_0603_1608Metric
- removed L2: 4.7uH, Inductor_SMD:L_Changjiang_FXL0630
- removed PS2: SY8113BADC, Thundergeddon:SOT95P285X100-6N
- removed R18: 118kΩ, Resistor_SMD:R_0603_1608Metric
- removed R19: 16.2kΩ, Resistor_SMD:R_0603_1608Metric
- added C24: 10uF, Capacitor_SMD:C_0805_2012Metric, F.Cu at (120.2, 39.7)
- added C25: 100nF, Capacitor_SMD:C_0805_2012Metric, F.Cu at (120.2, 42.7)
- added FB2: FerriteBead, Inductor_SMD:L_0603_1608Metric, F.Cu at (113.9, 54.8)
- added J3: Conn_01x02, Connector_PinHeader_2.54mm:PinHeader_1x02_P2.54mm_Vertical, F.Cu at (71.2, 80.5)
- added J4: Conn_01x03, Connector_PinHeader_2.54mm:PinHeader_1x03_P2.54mm_Vertical, F.Cu at (58.3, 77.9)
- added J5: Conn_01x02, Connector_PinHeader_2.54mm:PinHeader_1x02_P2.54mm_Vertical, F.Cu at (74.9, 80.4)
- added Q1: MMBT3904, Package_TO_SOT_SMD:SOT-23, F.Cu at (118.3, 55.7)
- added R10: 100kΩ, Resistor_SMD:R_0603_1608Metric, F.Cu at (113.9, 57.3)
- added R11: 220Ω, Resistor_SMD:R_0402_1005Metric, F.Cu at (105.8, 47.2)
- added R12: 220Ω, Resistor_SMD:R_0402_1005Metric, F.Cu at (105.8, 49.2)
- added R6: 5.1 kΩ, Resistor_SMD:R_0402_1005Metric, F.Cu at (105.8, 39.2)
- added R7: 5.1 kΩ, Resistor_SMD:R_0402_1005Metric, F.Cu at (105.8, 41.2)
- added R8: 330Ω, Resistor_SMD:R_0402_1005Metric, F.Cu at (105.8, 43.2)
- added R9: 1k, Resistor_SMD:R_0402_1005Metric, F.Cu at (105.8, 45.2)
- C11: value 47uF -> 1uF; footprint Capacitor_SMD:C_0805_2012Metric -> Capacitor_SMD:C_0201_0603Metric
- C12: value 10uF -> 220uF; footprint Capacitor_SMD:C_0805_2012Metric -> Capacitor_SMD:CP_Elec_6.3x5.4
- C8: footprint Capacitor_SMD:C_0603_1608Metric -> Capacitor_SMD:C_0402_1005Metric
- J6: renamed from P1; value USB_C_Plug -> USB_C_Receptacle_USB2.0_16P
- moved C8 36.5 mm to (119.4, 45.2)
- moved C11 34.1 mm to (108.5, 56.9)
- moved C12 29.3 mm to (65.0, 89.5)
- moved J2 3.59 mm to (72.2, 74.4), turned to 180 degrees
- moved L1 1.02 mm to (79.2, 90.7)
- turned U1 to 90 degrees
Connections:
- net CAM_1V2 renamed +CAM_1V2
- net Net-(J2-AVDD) renamed +CAM_AVDD_3V3
- BZ1 pad 1: unconnected-(BZ1-+-Pad1) -> +3V3
- BZ1 pad 2: unconnected-(BZ1---Pad2) -> Net-(BZ1--)
- C11 pad 1: +5V -> +3V3_CLEAN
- C12 pad 2: +BATT -> +3V3
- C18 pad 2: +3V3 -> +3V3_CLEAN
- C19 pad 2: +3V3 -> +3V3_CLEAN
- C20 pad 2: +3V3 -> +3V3_CLEAN
- C21 pad 2: +3V3 -> +3V3_CLEAN
- C8 pad 1: +5V -> +3V3_CLEAN
- FB1 pad 1: +3V3 -> +3V3_CLEAN
- J1 pad 1: unconnected-(J1-Pin_1-Pad1) -> +BATT
- J1 pad 2: unconnected-(J1-Pin_2-Pad2) -> GND
- J1 pad 3: unconnected-(J1-Pin_3-Pad3) -> /I2C SDA
- J1 pad 4: unconnected-(J1-Pin_4-Pad4) -> /I2C SCL
- J6 pad A12: Net-(P1-GND-PadA1) -> GND
- J6 pad A5: unconnected-(P1-CC-PadA5) -> Net-(J6-CC1)
- J6 pad A9: Net-(P1-VBUS-PadA4) -> +BATT
- J6 pad B12: Net-(P1-GND-PadA1) -> GND
- J6 pad B5: unconnected-(P1-VCONN-PadB5) -> Net-(J6-CC2)
- J6 pad B9: Net-(P1-VBUS-PadA4) -> +BATT
- J6 pad S1: unconnected-(P1-SHIELD-PadS1) -> GND
- U1 pad 1: Net-(U1-GND-Pad1) -> GND
- U1 pad 10: unconnected-(U1-GPIO17/U1TXD/ADC2_CH6-Pad10) -> /GPIO17
- U1 pad 11: unconnected-(U1-GPIO18/U1RXD/ADC2_CH7/CLK_OUT3-Pad11) -> /GPIO18
- U1 pad 12: unconnected-(U1-GPIO8/TOUCH8/ADC1_CH7/SUBSPICS1-Pad12) -> /GPIO8
- U1 pad 13: unconnected-(U1-GPIO19/U1RTS/ADC2_CH8/CLK_OUT2/USB_D--Pad13) -> USB_D+
- U1 pad 14: unconnected-(U1-GPIO20/U1CTS/ADC2_CH9/CLK_OUT1/USB_D+-Pad14) -> USB_D-
- U1 pad 17: unconnected-(U1-GPIO9/TOUCH9/ADC1_CH8/FSPIHD/SUBSPIHD-Pad17) -> /GPIO9
- U1 pad 18: unconnected-(U1-GPIO10/TOUCH10/ADC1_CH9/FSPICS0/FSPIIO4/SUBSPICS0-Pad18) -> /GPIO10
- U1 pad 19: unconnected-(U1-GPIO11/TOUCH11/ADC2_CH0/FSPID/FSPIIO5/SUBSPID-Pad19) -> /GPIO11
- U1 pad 2: unconnected-(U1-3V3-Pad2) -> +3V3_CLEAN
- U1 pad 20: unconnected-(U1-GPIO12/TOUCH12/ADC2_CH1/FSPICLK/FSPIIO6/SUBSPICLK-Pad20) -> /GPIO12
- U1 pad 21: unconnected-(U1-GPIO13/TOUCH13/ADC2_CH2/FSPIQ/FSPIIO7/SUBSPIQ-Pad21) -> /GPIO13
- U1 pad 23: unconnected-(U1-GPIO21-Pad23) -> /I2C SDA
- U1 pad 24: unconnected-(U1-GPIO47/SPICLK_P/SUBSPICLK_P_DIFF-Pad24) -> /I2C SCL
- U1 pad 31: unconnected-(U1-GPIO38/FSPIWP/SUBSPIWP-Pad31) -> /STATUS_LEDS
- U1 pad 32: unconnected-(U1-MTCK/GPIO39/CLK_OUT3/SUBSPICS1-Pad32) -> /IR #1
- U1 pad 33: unconnected-(U1-MTDO/GPIO40/CLK_OUT2-Pad33) -> /IR #2
- U1 pad 4: unconnected-(U1-GPIO4/TOUCH4/ADC1_CH3-Pad4) -> /GPIO4
- U1 pad 40: Net-(U1-GND-Pad1) -> GND
- U1 pad 41: Net-(U1-GND-Pad1) -> GND
- U1 pad 5: unconnected-(U1-GPIO5/TOUCH5/ADC1_CH4-Pad5) -> /GPIO5
- U1 pad 6: unconnected-(U1-GPIO6/TOUCH6/ADC1_CH5-Pad6) -> /GPIO6
- U1 pad 7: unconnected-(U1-GPIO7/TOUCH7/ADC1_CH6-Pad7) -> /GPIO7
- U1 pad 8: unconnected-(U1-GPIO15/U0RTS/ADC2_CH4/XTAL_32K_P-Pad8) -> /GPIO15
- U1 pad 9: unconnected-(U1-GPIO16/U0CTS/ADC2_CH5/XTAL_32K_N-Pad9) -> /GPIO16
- U2 pad 1: +3V3 -> +3V3_CLEAN
- U2 pad 3: +3V3 -> +3V3_CLEAN
- U4 pad 1: +3V3 -> +3V3_CLEAN
- U4 pad 3: +3V3 -> +3V3_CLEAN

Commit message: Signed-off-by: SMAUG\Pete <pwbrophy@gmail.com>
Parts:
- added C22: 100nF, Capacitor_SMD:C_0402_1005Metric, F.Cu at (42.1, 56.0)
- added C23: 1.0uF, Capacitor_SMD:C_0603_1608Metric, F.Cu at (42.7, 49.7)
- added R15: 10k, Resistor_SMD:R_0402_1005Metric, F.Cu at (42.1, 52.0)
- added R16: 10k, Resistor_SMD:R_0402_1005Metric, F.Cu at (42.1, 54.0)
- added SW1: SW_Push, Button_Switch_SMD:SW_SPST_TL3342, B.Cu at (70.2, 46.0)
- added SW2: SW_Push, Button_Switch_SMD:SW_SPST_TL3342, B.Cu at (60.6, 45.9)
- CON_IR_LED_1: renamed from J3; moved to B.Cu
- CON_IR_LED_2: renamed from J5; moved to B.Cu
- J1: footprint Connector_JST:JST_XH_B4B-XH-A_1x04_P2.50mm_Vertical -> Connector_JST:JST_XH_S4B-XH-A_1x04_P2.50mm_Horizontal
- U1: value ESP32-WROVER-E -> ESP32-S3-WROOM-1; footprint RF_Module:ESP32-S3-WROOM-1U -> PCM_Espressif:ESP32-S3-WROOM-1U
- moved J1 9.29 mm to (85.9, 69.0), turned to 90 degrees
- moved CON_IR_LED_1 7.02 mm to (64.2, 81.4), turned to -90 degrees
- moved CON_STATUS_LED1 4.93 mm to (58.0, 82.8), turned to 180 degrees
- moved R1 4.53 mm to (109.7, 41.6)
- moved R2 4.53 mm to (109.7, 43.6)
- moved BZ1 4.22 mm to (82.7, 57.2)
- moved U1 4.03 mm to (65.3, 58.7), turned to 0 degrees
- moved C18 3.64 mm to (61.4, 88.7), turned to 90 degrees
- moved L1 2.58 mm to (80.0, 93.1)
- moved J3 2.09 mm to (71.4, 76.3), turned to 0 degrees
- moved CON_IR_LED_2 1.57 mm to (76.0, 81.5), turned to -90 degrees
- renumbered C25 to C1, C4 to C10, C6 to C11, C5 to C12, C1 to C13, C17 to C14, C2 to C15, C3 to C16, C20 to C17, C12 to C18, C18 to C19, C24 to C2, C21 to C20, C19 to C21, C7 to C3, C9 to C4, C10 to C5, C13 to C6, C14 to C7, C11 to C9, J4 to CON_STATUS_LED1, FB2 to FB1, FB1 to FB2, J6 to J2, J2 to J3, R6 to R1, R3 to R10, R5 to R11, R4 to R12, R1 to R13, R8 to R14, R7 to R2, R15 to R3, R16 to R4, R11 to R5, R12 to R6, R2 to R7, R9 to R8, R10 to R9, U4 to U3
Connections:
- U1 pad 13: USB_D+ -> USB_D-
- U1 pad 14: USB_D- -> USB_D+
- U1 pad 27: unconnected-(U1-GPIO0/BOOT-Pad27) -> Net-(U1-GPIO0/BOOT)
- U1 pad 3: unconnected-(U1-EN-Pad3) -> Net-(U1-EN)
Routing:
- net /GPIO18: track 0.00 -> 19.9 mm, vias 0 -> 2
- net /GPIO9: track 0.00 -> 9.91 mm
- net /GPIO10: track 0.00 -> 9.34 mm
- net /GPIO11: track 0.00 -> 8.68 mm
- net /GPIO12: track 0.00 -> 8.36 mm
- net /GPIO13: track 0.00 -> 8.04 mm

Commit message: Signed-off-by: SMAUG\Pete <pwbrophy@gmail.com>
Parts:
- added D1: D_Schottky, Diode_SMD:D_SOD-123, B.Cu at (83.2, 52.6)
- C22, C23, R15, R16: moved to B.Cu
- J2: footprint Connector_USB:USB_C_Receptacle_HRO_TYPE-C-31-M-17 -> Connector_USB:USB_C_Receptacle_HRO_TYPE-C-31-M-12
- moved C8 74.3 mm to (84.8, 111.0)
- moved C9 66.9 mm to (73.8, 114.1)
- moved FB1 66.9 mm to (79.2, 111.9)
- moved R14 57.1 mm to (61.0, 78.6)
- moved R5 56.3 mm to (61.4, 81.7)
- moved C7 54.0 mm to (79.1, 109.0)
- moved R4 50.8 mm to (78.1, 119.6)
- moved R6 46.2 mm to (76.1, 84.5)
- moved U2 45.6 mm to (70.9, 70.5), turned to -90 degrees
- moved U3 42.0 mm to (75.1, 70.6), turned to -90 degrees
- moved C1 36.5 mm to (84.1, 37.2)
- moved C2 36.5 mm to (84.1, 34.2)
- moved Q1 36.0 mm to (82.3, 54.2), turned to 180 degrees
- moved C4 34.8 mm to (75.2, 89.0)
- moved R9 34.2 mm to (79.7, 56.8)
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Connections:
- C1 pad 1: +BATT -> +5V_USB
- C2 pad 1: +BATT -> +5V_USB
- J2 pad A9: +BATT -> +5V_USB
- J2 pad B9: +BATT -> +5V_USB
Routing:
- net /GPIO18: track 19.9 -> 0.00 mm, vias 2 -> 0
- net /GPIO9: track 9.91 -> 0.00 mm
- net /GPIO10: track 9.34 -> 0.00 mm
- net /GPIO11: track 8.68 -> 0.00 mm
- net /GPIO12: track 8.36 -> 0.00 mm
- net /GPIO13: track 8.04 -> 0.00 mm

Commit message: Signed-off-by: SMAUG\Pete <pwbrophy@gmail.com>
Parts:
- J3: footprint Connector_FFC-FPC:TE_2-1734839-4_1x24-1MP_P0.5mm_Horizontal -> Jushuo:AFC07-S24ECA-00
- moved CON_STATUS_LED1 6.64 mm to (63.6, 86.5), turned to -90 degrees
- moved C18 5.53 mm to (65.0, 92.9)
- moved U3 3.47 mm to (78.2, 68.8), turned to 0 degrees
- moved CON_IR_LED_2 2.95 mm to (78.8, 82.6), turned to 90 degrees
- moved U2 1.60 mm to (70.4, 69.0), turned to 0 degrees
- moved CON_IR_LED_1 1.22 mm to (63.7, 82.5)
- moved J3 0.05 mm to (71.3, 76.3)

Commit message: Signed-off-by: SMAUG\Pete <pwbrophy@gmail.com>
Parts:
- added C24: 22uF, Capacitor_SMD:C_0805_2012Metric, F.Cu at (62.2, 91.0)
- added C25: 100nF, Capacitor_SMD:C_0603_1608Metric, F.Cu at (62.4, 89.1)
- C18: value 220uF -> 22uF; footprint Capacitor_SMD:CP_Elec_6.3x5.4 -> Capacitor_SMD:C_0805_2012Metric
- J3: footprint Jushuo:AFC07-S24ECA-00 -> Jushuo:AFC07-S24ECA-00_flux
- SW1, SW2: footprint Button_Switch_SMD:SW_SPST_TL3342 -> Button_Switch_SMD:SW_Push_1P1T_XKB_TS-1187A
- moved C18 2.69 mm to (62.3, 93.2), turned to 0 degrees
- moved CON_IR_LED_1 0.40 mm to (63.7, 82.9)
- moved CON_IR_LED_2 0.30 mm to (78.8, 82.9)
- moved BZ1 0.21 mm to (86.1, 54.0)

Commit message: Signed-off-by: SMAUG\Pete <pwbrophy@gmail.com>
Parts:
- removed U2: TLV70028_SOT353, Package_TO_SOT_SMD:SOT-23-5
- added U4: LN1234B132MR-G, Package_TO_SOT_SMD:SOT-23-5, F.Cu at (74.2, 69.9)
- C13: value 100nF -> 4.7uF; footprint Capacitor_SMD:C_0402_1005Metric -> Capacitor_SMD:C_0201_0603Metric
- C15: value 1uF -> 100nF; footprint Capacitor_SMD:C_0201_0603Metric -> Capacitor_SMD:C_0402_1005Metric
- C16: value 4.7uF -> 1uF; footprint Capacitor_SMD:C_0805_2012Metric -> Capacitor_SMD:C_0201_0603Metric
- U3: value TLV70012_SOT23-5 -> ME6211C28M5G
- moved C16 16.2 mm to (101.4, 68.6)
- moved FB2 16.1 mm to (104.6, 67.3)
- moved U3 8.63 mm to (69.6, 69.9)
- moved C13 5.98 mm to (101.4, 66.9)
- moved C15 3.32 mm to (104.0, 69.5)
Connections:
- C11 pad 2: +CAM_1V2 -> +CAM_1V3
- C13 pad 1: +CAM_AVDD_3V3 -> GND
- C13 pad 2: GND -> +CAM_2V8
- C14 pad 2: +CAM_1V2 -> +CAM_1V3
- C15 pad 1: +CAM_AVDD_3V3 -> +CAM_AVDD_2V8
- C16 pad 1: +CAM_AVDD_3V3 -> +CAM_AVDD_2V8
- FB2 pad 1: +3V3_CLEAN -> +CAM_AVDD_2V8
- FB2 pad 2: +CAM_AVDD_3V3 -> +CAM_2V8
- J3 pad 15: +CAM_1V2 -> +CAM_1V3
- J3 pad 21: +CAM_AVDD_3V3 -> +CAM_AVDD_2V8
- U3 pad 5: +CAM_1V2 -> +CAM_2V8

Commit message: Signed-off-by: SMAUG\Pete <pwbrophy@gmail.com>
Parts:
- removed J3: Camera, Jushuo:AFC07-S24ECA-00_flux
- added C26: 100nF, Capacitor_SMD:C_0603_1608Metric, F.Cu at (97.0, 51.3)
- added D2: PRTR5V0U2X, Package_TO_SOT_SMD:SOT-143, F.Cu at (82.0, 45.2)
- added D3: LED, LED_SMD:LED_0603_1608Metric, F.Cu at (78.1, 105.3)
- added D4: LED, LED_SMD:LED_0805_2012Metric, F.Cu at (64.9, 105.1)
- added FPC1: AFC07-S24ECA-00, EasyEDA2Kicad:FPC-SMD_AFC07-S24ECA-00, F.Cu at (71.3, 76.3)
- added R17: 10k, Resistor_SMD:R_0603_1608Metric, F.Cu at (74.6, 105.3)
- added R18: 1k, Resistor_SMD:R_0603_1608Metric, F.Cu at (68.4, 105.0)
- C1: footprint Capacitor_SMD:C_0805_2012Metric -> Capacitor_SMD:C_0603_1608Metric
- C10, C11, C15, C17, C19, C22, C8: footprint Capacitor_SMD:C_0402_1005Metric -> Capacitor_SMD:C_0603_1608Metric
- C12, C14, C16, C20, C21, C9: footprint Capacitor_SMD:C_0201_0603Metric -> Capacitor_SMD:C_0603_1608Metric
- C13: footprint Capacitor_SMD:C_0201_0603Metric -> Capacitor_SMD:C_0805_2012Metric
- C23: value 1.0uF -> 1uF
- R1, R10, R11, R12, R13, R14, R15, R16, R2, R5, R6, R7, R8: footprint Resistor_SMD:R_0402_1005Metric -> Resistor_SMD:R_0603_1608Metric
- moved Q1 49.8 mm to (96.0, 102.2)
- moved FB2 41.8 mm to (62.9, 70.4)
- moved C16 38.8 mm to (62.7, 72.0)
- moved C15 38.0 mm to (66.1, 72.3), turned to 180 degrees
- moved BZ1 37.3 mm to (96.1, 89.9), turned to -90 degrees
- moved R13 35.9 mm to (61.9, 68.4)
- moved R7 34.9 mm to (62.6, 73.6)
- moved C12 33.9 mm to (69.3, 71.3), turned to 180 degrees
- moved C13 32.6 mm to (68.8, 69.2), turned to 180 degrees
- moved R10 32.3 mm to (66.0, 69.9), turned to -90 degrees
- moved C10 31.3 mm to (69.2, 72.9)
- moved C21 30.3 mm to (75.1, 66.3)
- moved C19 29.0 mm to (75.2, 64.5)
- moved C20 28.3 mm to (78.2, 66.2)
- moved C14 28.3 mm to (75.6, 69.3)
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- renumbered CON_IR_LED_1 to J4, CON_IR_LED_2 to J5, CON_STATUS_LED1 to J6
Connections:
- net +5V_USB renamed /+5V_USB
- net USB_D+ renamed /USB_D+
- net USB_D- renamed /USB_D-
- R15 pad 1: +3V3_CLEAN -> +3V3
- R16 pad 1: +3V3_CLEAN -> +3V3
- U1 pad 2: +3V3_CLEAN -> +3V3
- U1 pad 25: unconnected-(U1-GPIO48/SPICLK_N/SUBSPICLK_N_DIFF-Pad25) -> /GPIO48
