File: TankTurret/TankTurret.kicad_pcb (KiCad board)
At the start: 2 copper layers, 35 x 60 mm, 65 parts, among them J1 Conn_01x04_Socket, J2 USB_C_Receptacle_USB2.0_16P, J4 Conn_01x02, J5 Conn_01x02, J6 Conn_01x03, Q1 MMBT3904, SW1 SW_Push, SW2 SW_Push, U1 ESP32-S3-WROOM-1, U3 ME6211C28M5G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

Commit message: Signed-off-by: SMAUG\Pete <pwbrophy@gmail.com>
Parts:
- C10, C11, C17, C19: footprint Capacitor_SMD:C_0603_1608Metric -> Capacitor_SMD:C_0402_1005Metric
- C22, C23, D1, R15, R16, SW1, SW2: moved to F.Cu
- J2: footprint Connector_USB:USB_C_Receptacle_HRO_TYPE-C-31-M-12 -> EasyEDA2Kicad:USB-C_SMD-TYPE-C-31-M-12_1; moved to F.Cu
- J6: moved to B.Cu
- moved R8 74.1 mm to (99.9, 104.3)
- moved R9 50.1 mm to (100.6, 102.4)
- moved J6 28.3 mm to (85.1, 76.3), turned to 0 degrees
- moved C25 27.9 mm to (84.8, 79.3), turned to 90 degrees
- moved C24 25.8 mm to (82.6, 74.1), turned to 90 degrees
- moved C17 24.0 mm to (77.3, 88.2), turned to 90 degrees
- moved C18 23.3 mm to (79.7, 73.4)
- moved C19 23.1 mm to (61.0, 82.7)
- moved C21 23.0 mm to (60.5, 84.1)
- moved R14 22.8 mm to (82.5, 70.7)
- moved C20 22.5 mm to (78.7, 88.7), turned to 90 degrees
- moved C13 21.5 mm to (82.0, 86.2)
- moved U3 20.3 mm to (78.4, 85.0), turned to 90 degrees
- moved C26 20.0 mm to (77.0, 51.8), turned to 90 degrees
- moved C2 19.7 mm to (84.7, 53.9), turned to -90 degrees
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Connections:
- FPC1 pad 12: /GPIO16 -> /GPIO15
- FPC1 pad 17: /GPIO13 -> /GPIO8
- FPC1 pad 18: /GPIO12 -> /GPIO9
- FPC1 pad 19: /GPIO11 -> /GPIO10
- FPC1 pad 20: /GPIO10 -> /GPIO11
- FPC1 pad 21: /GPIO9 -> /GPIO12
- FPC1 pad 22: /GPIO8 -> /GPIO13
- R1 pad 1: Net-(J2-CC1) -> Net-(J2-CC2)
- R11 pad 1: /GPIO15 -> /GPIO16
- R2 pad 1: Net-(J2-CC2) -> Net-(J2-CC1)
Routing:
- net +BATT: track 0.00 -> 59.4 mm
- net +3V3: track 0.00 -> 58.1 mm
- net +CAM_2V8: track 0.00 -> 40.0 mm, vias 0 -> 3
- net +3V3_CLEAN: track 0.00 -> 35.6 mm
- net /USB_D-: track 0.00 -> 27.3 mm
- net /USB_D+: track 0.00 -> 26.9 mm
- net GND: track 0.00 -> 26.4 mm, vias 0 -> 39
- net /GPIO13: track 0.00 -> 22.6 mm, vias 0 -> 2
- net /GPIO12: track 0.00 -> 21.1 mm, vias 0 -> 2
- net /GPIO11: track 0.00 -> 19.6 mm, vias 0 -> 2
- net /GPIO10: track 0.00 -> 18.0 mm, vias 0 -> 2
- net +CAM_AVDD_2V8: track 0.00 -> 16.8 mm
- net /GPIO9: track 0.00 -> 16.3 mm, vias 0 -> 2
- net /GPIO4: track 0.00 -> 14.3 mm
- net +CAM_1V3: track 0.00 -> 14.3 mm, vias 0 -> 2
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- added copper zone on F.Cu, net GND

Commit message: Signed-off-by: SMAUG\Pete <pwbrophy@gmail.com>
Parts:
- removed BZ1: Buzzer, Buzzer_Beeper:Buzzer_12x9.5RM7.6
- added J3: Conn_01x02, Connector_PinHeader_2.54mm:PinHeader_1x02_P2.54mm_Vertical, F.Cu at (57.5, 81.5)
- added R19: 4.7k, Resistor_SMD:R_0603_1608Metric, F.Cu at (77.2, 58.0)
- added R20: 4.7k, Resistor_SMD:R_0603_1608Metric, F.Cu at (79.8, 56.5)
- moved R8 54.7 mm to (56.1, 71.5), turned to 90 degrees
- moved R9 49.7 mm to (59.4, 74.7), turned to -90 degrees
- moved Q1 42.2 mm to (57.0, 75.2), turned to -90 degrees
- moved C23 26.0 mm to (58.0, 70.7)
- moved R2 14.9 mm to (82.9, 51.6), turned to -90 degrees
- moved SW2 12.1 mm to (59.5, 44.8)
- moved SW1 11.3 mm to (70.5, 44.8)
- moved R15 10.3 mm to (75.2, 43.3)
- moved C22 8.92 mm to (75.2, 46.3)
- moved C18 6.09 mm to (84.8, 70.2)
- moved J6 3.55 mm to (84.9, 72.8), turned to 90 degrees
- moved R1 3.42 mm to (79.7, 50.6), turned to 180 degrees
- moved C24 2.87 mm to (84.8, 76.0)
- moved J5 2.85 mm to (82.2, 77.3), turned to 180 degrees
- moved J4 2.46 mm to (60.5, 78.0), turned to 180 degrees
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Connections:
- U1 pad 32: /IR #1 -> /IR #2
- U1 pad 33: /IR #2 -> /IR #1
Routing:
- net +3V3: track 58.1 -> 118.5 mm, vias 0 -> 3
- net Net-(U1-EN): track 0.00 -> 39.7 mm, vias 0 -> 4
- net /IR #1: track 0.00 -> 28.2 mm, vias 0 -> 2
- net /BUZZER: track 0.00 -> 22.5 mm, vias 0 -> 2
- net Net-(U1-GPIO0/BOOT): track 0.00 -> 11.8 mm
- net /+5V_USB: track 7.33 -> 15.9 mm
- net GND: track 26.4 -> 33.9 mm, vias 39 -> 46
- net Net-(Q1-B): track 0.00 -> 4.74 mm
- net Net-(J3-Pin_2): track 0.00 -> 2.98 mm
- net /USB_D-: track 27.3 -> 30.2 mm, vias 0 -> 2
- net unconnected-(J2-SBU2-PadB8): track 2.31 -> 0.00 mm
- net Net-(J2-CC1): track 0.00 -> 2.04 mm
- net Net-(J2-CC2): track 0.00 -> 1.98 mm
- net /I2C SDA: track 14.1 -> 15.2 mm
- net /I2C SCL: track 13.5 -> 14.6 mm

Commit message: Signed-off-by: SMAUG\Pete <pwbrophy@gmail.com>
Parts:
- added TP1: TestPoint, TestPoint:TestPoint_Pad_D1.0mm, B.Cu at (62.9, 93.3)
- added TP10: TestPoint, TestPoint:TestPoint_Pad_D1.0mm, B.Cu at (72.7, 78.0)
- added TP11: TestPoint, TestPoint:TestPoint_Pad_D1.0mm, B.Cu at (72.2, 50.8)
- added TP12: TestPoint, TestPoint:TestPoint_Pad_D1.0mm, B.Cu at (74.2, 50.7)
- added TP13: TestPoint, TestPoint:TestPoint_Pad_D1.0mm, B.Cu at (57.1, 76.2)
- added TP14: TestPoint, TestPoint:TestPoint_Pad_D1.0mm, B.Cu at (63.4, 76.5)
- added TP15: TestPoint, TestPoint:TestPoint_Pad_D1.0mm, B.Cu at (79.3, 77.3)
- added TP16: TestPoint, TestPoint:TestPoint_Pad_D1.0mm, B.Cu at (79.7, 70.1)
- added TP2: TestPoint, TestPoint:TestPoint_Pad_D1.0mm, B.Cu at (70.5, 86.3)
- added TP3: TestPoint, TestPoint:TestPoint_Pad_D1.0mm, B.Cu at (81.5, 92.0)
- added TP4: TestPoint, TestPoint:TestPoint_Pad_D1.0mm, B.Cu at (69.0, 75.9)
- added TP5: TestPoint, TestPoint:TestPoint_Pad_D1.0mm, B.Cu at (68.7, 80.1)
- added TP6: TestPoint, TestPoint:TestPoint_Pad_D1.0mm, B.Cu at (66.6, 97.5)
- added TP6: TestPoint, TestPoint:TestPoint_Pad_D1.0mm, B.Cu at (70.8, 46.2)
- added TP7: TestPoint, TestPoint:TestPoint_Pad_D1.0mm, B.Cu at (81.3, 44.7)
- added TP8: TestPoint, TestPoint:TestPoint_Pad_D1.0mm, B.Cu at (79.6, 46.2)
- added TP9: TestPoint, TestPoint:TestPoint_Pad_D1.0mm, B.Cu at (82.5, 46.4)
- moved R6 7.95 mm to (82.1, 75.0), turned to 180 degrees
- moved R16 1.13 mm to (65.0, 42.7), turned to 180 degrees
- moved C21 0.68 mm to (59.9, 84.2)
- moved C25 0.65 mm to (85.5, 79.3)
- moved C19 0.20 mm to (61.0, 82.5)
- moved C16 0.10 mm to (64.3, 72.3)
- moved R8 0.06 mm to (56.2, 71.5)
- moved C12 0.06 mm to (79.0, 82.7)
- turned D4 to 180 degrees
- turned R14 to 90 degrees
- turned R15 to -90 degrees
Routing:
- net +3V3: track 118.5 -> 180.5 mm, vias 3 -> 4
- net /GPIO48: track 0.00 -> 53.6 mm, vias 0 -> 6
- net /IR #2: track 0.00 -> 33.3 mm, vias 0 -> 2
- net /STATUS_LEDS: track 0.00 -> 30.2 mm, vias 0 -> 2
- net GND: track 33.9 -> 53.5 mm, vias 46 -> 59
- net Net-(J6-Pin_2): track 0.00 -> 6.08 mm, vias 0 -> 1
- net Net-(J5-Pin_1): track 0.00 -> 5.50 mm, vias 0 -> 1
- net +3V3_CLEAN: track 35.3 -> 40.8 mm, vias 0 -> 1
- net /I2C SDA: track 15.2 -> 20.5 mm, vias 2 -> 3
- net Net-(J4-Pin_1): track 0.00 -> 4.98 mm, vias 0 -> 1
- net /I2C SCL: track 14.6 -> 18.6 mm, vias 2 -> 3
- net Net-(FPC1-XCLK1): track 8.39 -> 11.9 mm, vias 0 -> 1
- net Net-(U1-GPIO0/BOOT): track 11.8 -> 14.9 mm
- net +BATT: track 59.4 -> 62.1 mm, vias 0 -> 1
- net /USB_D-: track 30.2 -> 32.7 mm, vias 2 -> 3
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Other:
- board text added: "+"
- board text added: "+3V3"
- board text added: "+3V3_CLEAN"
- board text added: "+BATT"
- board text added: "-"
- board text added: "1V3"
- board text added: "2V8"
- board text added: "3V3"
- board text added: "5V"
- board text added: "BOOT"
- board text added: "BUZZ"
- board text added: "CAMERA"
- board text added: "D+"
- board text added: "D-"
- board text added: "DIN"
- board text added: "EN"
- board text added: "GND"
- board text added: "I2C"
- board text added: "I2C SCL I2C SDA GND +BATT"
- board text added: "IR LED 1"
- board text added: "IR LED 2"
- board text added: "SCL"
- board text added: "SDA"
- board text added: "THUNDERGEDDON"
- board text added: "TOP LED"
- board text added: "USB"
- board text added: "XCLK"

Commit message: Signed-off-by: SMAUG\Pete <pwbrophy@gmail.com>
Parts:
- added C27: 100nF, Capacitor_SMD:C_0603_1608Metric, F.Cu at (55.9, 68.3)
- added C28: 10uF, Capacitor_SMD:C_0805_2012Metric, F.Cu at (55.9, 71.0)
- moved R8 1.46 mm to (57.6, 71.6)
- moved R7 1.40 mm to (61.2, 69.1)
- moved C23 1.20 mm to (59.1, 70.7)
- moved R13 1.05 mm to (62.8, 69.1)
- moved TP16 0.63 mm to (79.1, 70.3)
- moved R5 0.30 mm to (61.2, 74.8)
- moved R9 0.27 mm to (59.6, 74.8)
- moved Q1 0.20 mm to (57.1, 75.2)
- moved TP11 0.07 mm to (72.2, 50.7)
- moved J3 0.06 mm to (57.5, 81.5)
Routing:
- net GND: track 53.5 -> 55.5 mm, vias 59 -> 61
- net /GPIO5: track 12.5 -> 11.8 mm
- net Net-(Q1-B): track 4.74 -> 4.03 mm
- net Net-(J6-Pin_2): track 6.08 -> 6.60 mm

Commit message: Signed-off-by: SMAUG\Pete <pwbrophy@gmail.com>
Parts:
- moved C12 3.17 mm to (82.0, 83.6)
- moved C10 1.42 mm to (75.8, 83.8)
- moved C11 1.25 mm to (67.3, 84.2)
- moved C14 1.25 mm to (67.2, 86.3)
- moved U4 1.25 mm to (64.1, 85.3)
- moved C19 0.82 mm to (61.2, 83.3)
- moved FB2 0.74 mm to (75.5, 86.3)
- moved C21 0.40 mm to (59.9, 84.5)
- moved TP2 0.07 mm to (70.6, 86.3)
Routing:
- net +CAM_2V8: track 41.1 -> 44.8 mm
- net +CAM_AVDD_2V8: track 17.2 -> 18.5 mm
- net +CAM_1V3: track 15.6 -> 16.8 mm

Commit message: Signed-off-by: SMAUG\Pete <pwbrophy@gmail.com>
Changed lines of the file:
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@@
 		(tags "resistor")
 		(property "Reference" "R6"
-			(at 2.6 -0.05 0)
+			(at 1.05 1.05 0)
 			(layer "F.SilkS")
 			(effects
@@
 		(tags "Through hole pin header THT 1x02 2.54mm single row")
 		(property "Reference" "J5"
-			(at 2.05 -2.85 90)
+			(at 1.1 -4.7 90)
 			(layer "F.SilkS")
 			(effects
@@
 	)
 	(gr_text "BOOT"
-		(at 66.75 47.3 90)
+		(at 66.6 47.7 90)
 		(layer "F.SilkS" knockout)
 		(effects

Commit message: Signed-off-by: SMAUG\Pete <pwbrophy@gmail.com>
Parts:
- removed the TP6 at (66.6, 97.5)
- removed the TP6 at (70.8, 46.2)
- added C29: 22uF, Capacitor_SMD:C_0805_2012Metric, F.Cu at (82.9, 69.7)
- added R21: 33Ω, Resistor_SMD:R_0402_1005Metric, F.Cu at (76.7, 54.6)
- added R22: 33Ω, Resistor_SMD:R_0402_1005Metric, F.Cu at (77.5, 53.9)
- added TP6: TestPoint, TestPoint:TestPoint_Pad_D1.0mm, B.Cu at (66.5, 97.2)
- moved R2 5.23 mm to (84.2, 56.6), turned to 0 degrees
- moved C25 3.99 mm to (84.8, 75.4)
- moved C24 2.76 mm to (85.0, 78.7), turned to -90 degrees
- moved D2 2.10 mm to (81.8, 53.2), turned to 180 degrees
- moved TP12 2.05 mm to (72.2, 50.7)
- moved TP11 2.00 mm to (74.2, 50.7)
- moved TP16 1.96 mm to (77.2, 70.5)
- moved R14 1.16 mm to (81.0, 69.9)
- moved TP14 1.00 mm to (63.3, 77.5)
- moved C18 0.47 mm to (85.0, 69.7), turned to -90 degrees
- moved TP15 0.32 mm to (79.1, 77.2)
- moved TP2 0.07 mm to (70.5, 86.3)
Connections:
- TP11 pad 1: /I2C SCL -> Net-(U1-GPIO21)
- TP12 pad 1: /I2C SDA -> Net-(U1-GPIO47/SPICLK_P/SUBSPICLK_P_DIFF)
- U1 pad 23: /I2C SDA -> Net-(U1-GPIO21)
- U1 pad 24: /I2C SCL -> Net-(U1-GPIO47/SPICLK_P/SUBSPICLK_P_DIFF)
Routing:
- net /I2C SDA: track 20.5 -> 12.8 mm, vias 3 -> 2
- net Net-(U1-GPIO21): track 0.00 -> 7.67 mm, vias 0 -> 1
- net Net-(U1-GPIO47/SPICLK_P/SUBSPICLK_P_DIFF): track 0.00 -> 7.17 mm, vias 0 -> 1
- net /I2C SCL: track 18.6 -> 11.5 mm, vias 3 -> 2
- net Net-(J2-CC1): track 2.04 -> 8.15 mm
- net +3V3: track 180.5 -> 183.1 mm, vias 4 -> 5
- net /USB_D-: track 32.7 -> 30.8 mm, vias 3 -> 1
- net GND: track 55.0 -> 56.5 mm, vias 61 -> 62
- net Net-(J4-Pin_1): track 5.11 -> 5.67 mm, vias 1 -> 0

Commit message: Signed-off-by: SMAUG\Pete <pwbrophy@gmail.com>
Parts:
- removed TP9: TestPoint, TestPoint:TestPoint_Pad_D1.0mm
- moved TP8 8.60 mm to (71.0, 46.3)
- moved D2 1.65 mm to (81.8, 51.6)
- moved R1 1.12 mm to (79.4, 51.7), turned to -90 degrees
- moved C26 0.59 mm to (77.7, 51.1)
- moved R12 0.16 mm to (69.5, 72.1)
Connections:
- net /STATUS_LEDS renamed /WS2812_LEDS
- C26 pad 2: +3V3 -> /+5V_USB
- D2 pad 4: +3V3 -> /+5V_USB
- TP8 pad 1: /USB_D+ -> GND
Routing:
- net /+5V_USB: track 17.4 -> 24.3 mm
- net /USB_D+: track 29.2 -> 26.1 mm, vias 1 -> 0
- net +3V3: track 183.1 -> 180.8 mm, vias 5 -> 4
- net /USB_D-: track 30.8 -> 28.5 mm, vias 1 -> 0
- net GND: track 56.5 -> 57.5 mm
Other:
- board text removed: "D+"
- board text removed: "D-"
