File: TankTurret/TankTurret.kicad_pcb (KiCad board)
At the start: 2 copper layers, 35 x 60 mm, 87 parts, among them J1 Conn_01x04_Socket, J2 USB_C_Receptacle_USB2.0_16P, J3 Conn_01x02, J4 Conn_01x02, J5 Conn_01x02, J6 Conn_01x03, Q1 MMBT3904, SW1 SW_Push, SW2 SW_Push, U1 ESP32-S3-WROOM-1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

Commit message: Signed-off-by: SMAUG\Pete <pwbrophy@gmail.com>
Parts:
- removed C22: 100nF, Capacitor_SMD:C_0603_1608Metric
- added R23: 22Ω, Resistor_SMD:R_0402_1005Metric, F.Cu at (73.6, 68.3)
- added R24: 22Ω, Resistor_SMD:R_0402_1005Metric, F.Cu at (76.4, 65.5)
- added R25: 4.7k, Resistor_SMD:R_0603_1608Metric, F.Cu at (78.3, 57.8)
- J1: value Conn_01x04_Socket -> Conn_01x05_Socket; footprint Connector_JST:JST_XH_S4B-XH-A_1x04_P2.50mm_Horizontal -> Connector_JST:JST_PH_S5B-PH-K_1x05_P2.00mm_Horizontal
- R17: value 10k -> 2.2k
- moved R16 4.10 mm to (65.0, 46.8)
- moved R15 2.90 mm to (75.1, 46.2)
- moved R20 2.28 mm to (79.7, 54.2), turned to 0 degrees
- moved R19 2.06 mm to (78.3, 56.2), turned to 0 degrees
- moved TP14 1.10 mm to (64.4, 77.5)
- moved R22 1.00 mm to (76.6, 53.5), turned to 180 degrees
- turned R21 to 180 degrees
- turned SW2 to 0 degrees
Connections:
- J1 pad 2: GND -> /INT
- J1 pad 3: /I2C SDA -> GND
- J1 pad 4: /I2C SCL -> /I2C SDA
- U1 pad 13: /USB_D- -> /USB_D-_ESP32
- U1 pad 14: /USB_D+ -> /USB_D+_ESP32
- U1 pad 22: unconnected-(U1-GPIO14/TOUCH14/ADC2_CH3/FSPIWP/FSPIDQS/SUBSPIWP-Pad22) -> /INT
Routing:
- net /INT: track 0.00 -> 18.3 mm, vias 0 -> 2
- net Net-(U1-GPIO0/BOOT): track 14.9 -> 10.5 mm
- net /USB_D+: track 26.1 -> 21.7 mm
- net Net-(U1-EN): track 38.1 -> 33.8 mm
- net /USB_D+_ESP32: track 0.00 -> 3.41 mm
- net /USB_D-: track 28.5 -> 25.9 mm
- net /USB_D-_ESP32: track 0.00 -> 2.53 mm
- net +3V3: track 180.8 -> 178.9 mm
- net /IR #2: track 33.3 -> 34.6 mm
- net /GPIO12: track 21.0 -> 19.8 mm
- net /GPIO11: track 19.6 -> 18.3 mm
- net /GPIO10: track 18.0 -> 16.8 mm
- net /GPIO13: track 22.5 -> 21.3 mm
- net /I2C SCL: track 11.5 -> 12.6 mm
- net /GPIO9: track 16.3 -> 15.1 mm
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Other:
- board text added: "FLASH"
- board text added: "I2C SCL I2C SDA GND INT +BATT"
- board text added: "RESET"
- board text removed: "BOOT"
- board text removed: "EN"
- board text removed: "I2C SCL I2C SDA GND +BATT"

Commit message: V0.2 Files sent to JLC PCB on 15/03/2026
Parts:
- moved C24 0.37 mm to (84.6, 78.7)
- moved C28 0.33 mm to (56.2, 70.9)
- moved R7 0.29 mm to (61.5, 69.2)
- moved R13 0.29 mm to (63.0, 69.2)
- moved C23 0.28 mm to (59.4, 70.6)
- moved R8 0.28 mm to (57.9, 71.6)
- moved J3 0.18 mm to (57.6, 81.4)
- moved Q1 0.17 mm to (57.1, 75.1)
Routing:
- net +BATT: track 62.1 -> 64.7 mm
Other:
- board text added: "v0.2"
