File: TankTurret/TankTurret.kicad_sch (KiCad schematic)
At the start: 24 parts, among them J2 Camera, J3 SlipRing_6, P1 USB_C_Plug, U1 ESP32-WROVER-E

Commit message: camera connector
Parts:
- removed J3: SlipRing_6, Connector_JST:JST_XH_B6B-XH-A_1x06_P2.50mm_Vertical, symbol Connector_Generic:Conn_02x03_Odd_Even
- removed R17: 10kΩ, Resistor_SMD:R_0603_1608Metri, symbol Device:R
- added C1, C18, C20, C4, C6: 100nF, Capacitor_SMD:C_0402_1005Metric, symbol Device:C
- added C17, C19, C2, C21, C5: 1uF, Capacitor_SMD:C_0201_0603Metric, symbol Device:C
- added C3: 4.7uF, Capacitor_SMD:C_0805_2012Metric, symbol Device:C
- added FB1: FerriteBead, Inductor_SMD:L_0603_1608Metric, symbol Device:FerriteBead
- added J1: Conn_01x04_Socket, Connector_JST:JST_XH_B4B-XH-A_1x04_P2.50mm_Vertical, symbol Connector:Conn_01x04_Socket
- added R1, R2: 4.7k, Resistor_SMD:R_0402_1005Metric, symbol Device:R
- added R3, R4: 10k, Resistor_SMD:R_0402_1005Metric, symbol Device:R
- added R5: 33Ω, Resistor_SMD:R_0402_1005Metric, symbol Device:R
- added U2: TLV70028_SOT353, Package_TO_SOT_SMD:SOT-23-5, symbol Regulator_Linear:TLV70012_SOT23-5
- added U4: TLV70012_SOT23-5, Package_TO_SOT_SMD:SOT-23-5, symbol Regulator_Linear:TLV70012_SOT23-5
- J2: footprint Connector_FFC-FPC:TE_2-1734839-3_1x23-1MP_P0.5mm_Horizontal -> Connector_FFC-FPC:TE_2-1734839-4_1x24-1MP_P0.5mm_Horizontal
- U1: footprint PCM_Espressif:ESP32-WROVER-E -> RF_Module:ESP32-S3-WROOM-1U; symbol PCM_Espressif:ESP32-WROVER-E -> PCM_Espressif:ESP32-S3-WROOM-1
Connections:
- net +3V3: now also C18.2, C19.2, C20.2, C21.2, FB1.1, U2.1 (IN), U2.3 (EN), U4.1 (IN), U4.3 (EN)
- net BUZZER: now also U1.39 (GPIO1/TOUCH1/ADC1_CH0); no longer U1.13 (MTMS/GPIO14/ADC2_CH6)
- net GND: now also J2.23 (AGND), U1.40 (GND), U1.41 (GND), C1.2, C17.1, C18.1, C19.1, C2.2, C20.1, C21.1, C3.2, C4.1, C5.1, C6.1, R4.1, U2.2 (GND), U4.2 (GND); no longer J2.17 (PWDN), U1.15 (GND), U1.38 (GND), U1.39 (GND_THERMAL)
- net GPIO18: now also J2.9 (Y7/D5), U1.11 (GPIO18/U1RXD/ADC2_CH7/CLK_OUT3); no longer J2.3 (Y4/D2), U1.30 (GPIO18)
- net GPIO19: no longer J2.5 (Y5/D3), U1.31 (GPIO19)
- net GPIO21: no longer J2.12 (XCLK), U1.33 (GPIO21)
- net GPIO22: no longer J2.8 (PCLK), U1.36 (GPIO22)
- net GPIO23: no longer J2.16 (HREF/HSYNC), U1.37 (GPIO23)
- net GPIO25: no longer J2.18 (VSYNC), U1.10 (DAC_1/ADC2_CH8/GPIO25)
- net GPIO26: no longer J2.22 (SIO_D), U1.11 (DAC_2/ADC2_CH9/GPIO26)
- net GPIO27: no longer J2.20 (SIO_C), U1.12 (ADC2_CH7/GPIO27)
- net GPIO34: no longer J2.11 (Y8/D6), U1.6 (GPIO34/ADC1_CH6)
- net GPIO35: no longer J2.13 (Y9/D7), U1.7 (GPIO35/ADC1_CH7)
- net GPIO36: no longer J2.7 (Y6/D4), U1.4 (SENSOR_VP/GPIO36/ADC1_CH0)
- net GPIO39: no longer J2.9 (Y7/D5), U1.5 (SENSOR_VN/GPIO39/ADC1_CH3)
- net GPIO4: now also J2.22 (SIO_D), U1.4 (GPIO4/TOUCH4/ADC1_CH3), R2.2; no longer J2.6 (Y2/D0), U1.26 (ADC2_CH0/GPIO4)
- net GPIO5: now also J2.20 (SIO_C), U1.5 (GPIO5/TOUCH5/ADC1_CH4), R1.1; no longer J2.4 (Y3/D1), U1.29 (GPIO5)
- net I2C SCL: now also U1.24 (GPIO47/SPICLK_P/SUBSPICLK_P_DIFF); no longer U1.8 (32K_XP/GPIO32/ADC1_CH4)
- net I2C SDA: now also U1.23 (GPIO21); no longer U1.9 (32K_XN/GPIO33/ADC1_CH5)
- net IR #1: now also U1.32 (MTCK/GPIO39/CLK_OUT3/SUBSPICS1); no longer U1.14 (MTDI/GPIO12/ADC2_CH5)
- net IR #2: now also U1.33 (MTDO/GPIO40/CLK_OUT2); no longer U1.24 (ADC2_CH2/GPIO2)
- net TOP_LEDS: now also U1.31 (GPIO38/FSPIWP/SUBSPIWP); no longer U1.16 (MTCK/GPIO13/ADC2_CH4)
- net USB-UART RX: no longer U1.34 (U0RXD/GPIO3)
- net USB-UART TX: no longer U1.35 (U0TXD/GPIO1)
- net at J2.19 (RESETB): now also R3.2
- net +CAM_2V8: now reaches J2.14 (DOVDD)
- net +CAM_2V8: now also C4.2, C5.2, R1.2, R2.1, R3.1, U2.5 (OUT)
- net +CAM_1V2: now reaches J2.15 (DVDD)
- net +CAM_1V2: now also C17.2, C6.2, U4.5 (OUT)
- net +CAM_AVDD_3V3: now reaches J2.21 (AVDD)
- net +CAM_AVDD_3V3: now also C1.1, C2.1, C3.1, FB1.2
- new net: J2.17 (PWDN), R4.2
- new net: J2.12 (XCLK), R5.2
- new net GPIO10: J2.5 (Y5/D3), U1.18 (GPIO10/TOUCH10/ADC1_CH9/FSPICS0/FSPIIO4/SUBSPICS0)
- new net GPIO11: J2.6 (Y2/D0), U1.19 (GPIO11/TOUCH11/ADC2_CH0/FSPID/FSPIIO5/SUBSPID)
- new net GPIO12: J2.7 (Y6/D4), U1.20 (GPIO12/TOUCH12/ADC2_CH1/FSPICLK/FSPIIO6/SUBSPICLK)
- new net GPIO13: J2.8 (PCLK), U1.21 (GPIO13/TOUCH13/ADC2_CH2/FSPIQ/FSPIIO7/SUBSPIQ)
- new net GPIO15: R5.1, U1.8 (GPIO15/U0RTS/ADC2_CH4/XTAL_32K_P)
- new net GPIO16: J2.13 (Y9/D7), U1.9 (GPIO16/U0CTS/ADC2_CH5/XTAL_32K_N)
- new net GPIO17: J2.11 (Y8/D6), U1.10 (GPIO17/U1TXD/ADC2_CH6)
- new net GPIO6: J2.18 (VSYNC), U1.6 (GPIO6/TOUCH6/ADC1_CH5)
- new net GPIO7: J2.16 (HREF/HSYNC), U1.7 (GPIO7/TOUCH7/ADC1_CH6)
- new net GPIO8: J2.3 (Y4/D2), U1.12 (GPIO8/TOUCH8/ADC1_CH7/SUBSPICS1)
- new net GPIO9: J2.4 (Y3/D1), U1.17 (GPIO9/TOUCH9/ADC1_CH8/FSPIHD/SUBSPIHD)
- no-connect marks 2 -> 3
Other:
- moved on the sheet: BZ1, C10, C11, C12, C13, C14, C15, C16, C7, C8, C9, J2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

Commit message: bits
Parts:
- removed C15: 100nF, Capacitor_SMD:C_0603_1608Metric, symbol Device:C
- removed C16: 18pF, Capacitor_SMD:C_0603_1608Metric, symbol Device:C
- removed L2: 4.7uH, Inductor_SMD:L_Changjiang_FXL0630, symbol Device:L
- removed PS2: SY8113BADC, Thundergeddon:SOT95P285X100-6N, symbol SY8113BADC:SY8113BADC
- removed R18: 118kΩ, Resistor_SMD:R_0603_1608Metric, symbol Device:R
- removed R19: 16.2kΩ, Resistor_SMD:R_0603_1608Metric, symbol Device:R
- added C24: 10uF, Capacitor_SMD:C_0805_2012Metric, symbol Device:C
- added C25: 100nF, Capacitor_SMD:C_0805_2012Metric, symbol Device:C
- added FB2: FerriteBead, Inductor_SMD:L_0603_1608Metric, symbol Device:FerriteBead
- added J3, J5: Conn_01x02, Connector_PinHeader_2.54mm:PinHeader_1x02_P2.54mm_Vertical, symbol Connector_Generic:Conn_01x02
- added J4: Conn_01x03, Connector_PinHeader_2.54mm:PinHeader_1x03_P2.54mm_Vertical, symbol Connector_Generic:Conn_01x03
- added Q1: MMBT3904, Package_TO_SOT_SMD:SOT-23, symbol Transistor_BJT:MMBT3904
- added R10: 100kΩ, Resistor_SMD:R_0603_1608Metric, symbol Device:R
- added R11, R12: 220Ω, Resistor_SMD:R_0402_1005Metric, symbol Device:R
- added R6, R7: 5.1 kΩ, Resistor_SMD:R_0402_1005Metric, symbol Device:R
- added R8: 330Ω, Resistor_SMD:R_0402_1005Metric, symbol Device:R
- added R9: 1k, Resistor_SMD:R_0402_1005Metric, symbol Device:R
- C11: value 47uF -> 1uF; footprint Capacitor_SMD:C_0805_2012Metric -> Capacitor_SMD:C_0201_0603Metric; JLCPCB Part # C16780 -> (none); MANUFACTURER Samsung -> (none); Manufacturer_Part_Number C16780 -> (none)
- C12: value 10uF -> 220uF; footprint Capacitor_SMD:C_0805_2012Metric -> Capacitor_SMD:CP_Elec_6.3x5.4; JLCPCB Part # C15850 -> (none); MANUFACTURER Samsung -> (none); Manufacturer_Part_Number CL21A106KAYNNNE -> (none)
- C8: footprint Capacitor_SMD:C_0603_1608Metric -> Capacitor_SMD:C_0402_1005Metric; JLCPCB Part # C14663 -> (none); MANUFACTURER YAGEO -> (none); Manufacturer_Part_Number CC0603KRX7R9BB104 -> (none)
- J6: renamed from P1; value USB_C_Plug -> USB_C_Receptacle_USB2.0_16P; symbol Connector:USB_C_Plug -> Connector:USB_C_Receptacle_USB2.0_16P
Connections:
- net +5V is gone; now on net +3V3_CLEAN: C11.1, C8.1
- net +3V3: now also BZ1.1 (+), C12.2, FB2.2, J4.1 (Pin_1); no longer C18.2, C19.2, C20.2, C21.2, FB1.1, U2.1 (IN), U2.3 (EN), U4.1 (IN), U4.3 (EN)
- net +BATT: now also J1.1 (Pin_1), J6.A4 (VBUS), J6.A9 (VBUS), J6.B4 (VBUS), J6.B9 (VBUS), C24.1, C25.1; no longer C12.2
- net BUZZER: now also R9.2
- net GND: now also J1.2 (Pin_2), J6.A1 (GND), J6.A12 (GND), J6.B1 (GND), J6.B12 (GND), J6.S1 (SHIELD), C24.2, C25.2, J3.2 (Pin_2), J4.3 (Pin_3), J5.2 (Pin_2), Q1.2 (E), R10.1, R6.2, R7.2
- net I2C SCL: now also J1.4 (Pin_4)
- net I2C SDA: now also J1.3 (Pin_3)
- net IR #1: now also R11.2
- net IR #2: now also R12.2
- net at J6.A5 (CC1): now also R6.1
- net USB_D+: now reaches J6.A6 (D+)
- net USB_D+: now also J6.B6 (D+), U1.13 (GPIO19/U1RTS/ADC2_CH8/CLK_OUT2/USB_D-)
- net USB_D-: now reaches J6.A7 (D-)
- net USB_D-: now also J6.B7 (D-), U1.14 (GPIO20/U1CTS/ADC2_CH9/CLK_OUT1/USB_D+)
- net at J6.B5 (CC2): now also R7.1
- net at BZ1.2 (-): now also Q1.3 (C)
- net +3V3_CLEAN: now reaches U1.2 (3V3)
- net +3V3_CLEAN: now also C18.2, C19.2, C20.2, C21.2, FB1.1, U2.1 (IN), U2.3 (EN), U4.1 (IN), U4.3 (EN), FB2.1
- net TOP_LEDS renamed STATUS_LEDS
- net STATUS_LEDS: now also R8.2
- new net: J4.2 (Pin_2), R8.1
- new net: J5.1 (Pin_1), R12.1
- new net: Q1.1 (B), R10.2, R9.1
- new net: J3.1 (Pin_1), R11.1
- no-connect marks 3 -> 5
Other:
- note added: "Buzzer"
- note added: "IR LEDs"
- note added: "Status LEDs"
- note removed: "Buzzer and LEDs"
- note removed: "Convert Battery to 5V"
- moved on the sheet: BZ1, C1, C17, C18, C19, C2, C20, C21, C3, C4, C5, C6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

Commit message: Signed-off-by: SMAUG\Pete <pwbrophy@gmail.com>
Parts:
- added C22: 100nF, Capacitor_SMD:C_0402_1005Metric, symbol Device:C
- added C23: 1.0uF, Capacitor_SMD:C_0603_1608Metric, symbol Device:C
- added R15, R16: 10k, Resistor_SMD:R_0402_1005Metric, symbol Device:R
- added SW1, SW2: SW_Push, Button_Switch_SMD:SW_SPST_TL3342, symbol Switch:SW_Push
- CON_IR_LED_1: renamed from J3; now not fitted
- CON_IR_LED_2: renamed from J5; now not fitted
- CON_STATUS_LED1: renamed from J4; now not fitted
- U1: value ESP32-WROVER-E -> ESP32-S3-WROOM-1; footprint RF_Module:ESP32-S3-WROOM-1U -> PCM_Espressif:ESP32-S3-WROOM-1U; JLCPCB Part # C701352 -> (none); Manufacturer_Part_Number ESP32-WROVER-IE-N16R8 -> (none)
- renumbered C25 to C1, C4 to C10, C6 to C11, C5 to C12, C1 to C13, C17 to C14, C2 to C15, C3 to C16, C20 to C17, C12 to C18, C18 to C19, C24 to C2, C21 to C20, C19 to C21, C7 to C3, C9 to C4, C10 to C5, C13 to C6, C14 to C7, C11 to C9, FB2 to FB1, FB1 to FB2, J6 to J2, J2 to J3, R6 to R1, R3 to R10, R5 to R11, R4 to R12, R1 to R13, R8 to R14, R7 to R2, R15 to R3, R16 to R4, R11 to R5, R12 to R6, R2 to R7, R9 to R8, R10 to R9, U4 to U3
Connections:
- net +3V3_CLEAN: now also R15.1, R16.1
- net GND: now also C22.2, C23.1, SW1.2, SW2.1
- net USB_D+: now also U1.14 (GPIO20/U1CTS/ADC2_CH9/CLK_OUT1/USB_D+); no longer U1.13 (GPIO19/U1RTS/ADC2_CH8/CLK_OUT2/USB_D-)
- net USB_D-: now also U1.13 (GPIO19/U1RTS/ADC2_CH8/CLK_OUT2/USB_D-); no longer U1.14 (GPIO20/U1CTS/ADC2_CH9/CLK_OUT1/USB_D+)
- net at U1.27 (GPIO0/BOOT): now also C22.1, R15.2, SW1.1
- net at U1.3 (EN): now also C23.2, R16.2, SW2.2

Commit message: Signed-off-by: SMAUG\Pete <pwbrophy@gmail.com>
Parts:
- BZ1: now not fitted
- J1: footprint Connector_JST:JST_XH_B4B-XH-A_1x04_P2.50mm_Vertical -> Connector_JST:JST_XH_S4B-XH-A_1x04_P2.50mm_Horizontal
Other:
- note added: "Turret: Buzzer"
- note added: "Turret: Camera Connector"
- note added: "Turret: Convert Battery to 3.3V"
- note added: "Turret: ESP32"
- note added: "Turret: IR LEDs"
- note added: "Turret: Slip Ring Connector and Expansion Connections"
- note added: "Turret: Status LEDs"
- note added: "Turret: USB Connector"
- note removed: "Buzzer"
- note removed: "Camera Connector"
- note removed: "Convert Battery to 3.3V"
- note removed: "ESP32"
- note removed: "IR LEDs"
- note removed: "Slip Ring Connector and Expansion Connections"
- note removed: "Status LEDs"
- note removed: "USB Connector"
- moved on the sheet: C1, C2, C23, J2, R1, R2, SW2

Commit message: Signed-off-by: SMAUG\Pete <pwbrophy@gmail.com>
Parts:
- added D1: D_Schottky, Diode_SMD:D_SOD-123, symbol Device:D_Schottky
- J2: footprint Connector_USB:USB_C_Receptacle_HRO_TYPE-C-31-M-17 -> Connector_USB:USB_C_Receptacle_HRO_TYPE-C-31-M-12
Connections:
- net +BATT: now also D1.1 (K); no longer C1.1, C2.1, J2.A4 (VBUS), J2.A9 (VBUS), J2.B4 (VBUS), J2.B9 (VBUS)
- new net +5V_USB: C1.1, C2.1, D1.2 (A), J2.A4 (VBUS), J2.A9 (VBUS), J2.B4 (VBUS), J2.B9 (VBUS)
Other:
- moved on the sheet: C1, C2, J2, R1, R2

Commit message: Signed-off-by: SMAUG\Pete <pwbrophy@gmail.com>
Parts:
- removed U2: TLV70028_SOT353, Package_TO_SOT_SMD:SOT-23-5, symbol Regulator_Linear:TLV70012_SOT23-5
- removed U3: TLV70012_SOT23-5, Package_TO_SOT_SMD:SOT-23-5, symbol Regulator_Linear:TLV70012_SOT23-5
- added C24: 22uF, Capacitor_SMD:C_0805_2012Metric, symbol Device:C
- added C25: 100nF, Capacitor_SMD:C_0603_1608Metric, symbol Device:C
- added U3: ME6211C28M5G, Package_TO_SOT_SMD:SOT-23-5, symbol EasyEDA2Kicad:ME6211C28M5G
- added U4: LN1234B132MR-G, Package_TO_SOT_SMD:SOT-23-5, symbol EasyEDA2Kicad:LN1234B132MR-G
- C13: value 100nF -> 4.7uF; footprint Capacitor_SMD:C_0402_1005Metric -> Capacitor_SMD:C_0201_0603Metric
- C15: value 1uF -> 100nF; footprint Capacitor_SMD:C_0201_0603Metric -> Capacitor_SMD:C_0402_1005Metric
- C16: value 4.7uF -> 1uF; footprint Capacitor_SMD:C_0805_2012Metric -> Capacitor_SMD:C_0201_0603Metric
- C18: value 220uF -> 22uF; footprint Capacitor_SMD:CP_Elec_6.3x5.4 -> Capacitor_SMD:C_0805_2012Metric; JLCPCB Part # (none) -> C45783; Manufacturer_Name (none) -> Samsung; Manufacturer_Part_Number (none) -> CL21A226MAQNNNE
- C7: Notes (none) -> PS1:FB series to +3V3
- J1: JLCPCB Part # (none) -> C262643
- J2: JLCPCB Part # (none) -> C165948; Manufacturer_Name (none) -> Korean Hroparts Elec; Manufacturer_Part_Number (none) -> TYPE-C-31-M-12
- J3: footprint Connector_FFC-FPC:TE_2-1734839-4_1x24-1MP_P0.5mm_Horizontal -> Jushuo:AFC07-S24ECA-00_flux
- SW1, SW2: footprint Button_Switch_SMD:SW_SPST_TL3342 -> Button_Switch_SMD:SW_Push_1P1T_XKB_TS-1187A
- U1: JLCPCB Part # (none) -> C3013946; Manufacturer_Part_Number (none) -> ESP32-S3-WROOM-1U-N16R8
- renumbered CON_IR_LED_1 to J4, CON_IR_LED_2 to J5, CON_STATUS_LED1 to J6
Connections:
- net +3V3: now also C24.2, C25.2
- net +3V3_CLEAN: now also U3.1 (VIN), U3.3 (CE), U4.1 (VIN), U4.3 (CE); no longer FB2.1
- net +CAM_2V8: now also C13.2, FB2.2, U3.5 (VOUT)
- net GND: now also C13.1, C24.1, C25.1, U3.2 (VSS), U4.2 (VSS); no longer C13.2
- net +CAM_1V2 renamed +CAM_1V3
- net +CAM_1V3: now also U4.5 (VOUT)
- net +CAM_AVDD_3V3 renamed +CAM_AVDD_2V8
- net +CAM_AVDD_2V8: now also FB2.1; no longer C13.1, FB2.2
Other:
- note added: "DOVDD 2.8V DVDD 1.3V AVDD 2.8V"
- moved on the sheet: C10, C11, C12, C14, C17, C18, C19, C20, C21, J6, R10, R12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

Commit message: Signed-off-by: SMAUG\Pete <pwbrophy@gmail.com>
Parts:
- BZ1: Notes (none) -> 3V Piezo Buzzer
- C1, C2: Notes (none) -> J2:VBUS to +5V_USB decoupling to GND
- C10, C12, C13: Notes (none) -> U3:VOUT to DOVDD decoupling to GND
- C11, C14: Notes (none) -> U4:VOUT to DVDD decoupling to GND
- C15, C16: Notes (none) -> AVDD decoupling to +CAM_AVDD_28
- C17, C20: Notes (none) -> U3:VIN to +3V3_CLEAN decoupling to GND
- C18, C24, C25: Notes (none) -> J6:PIN1 to +3V3 decoupling to GND
- C19, C21: Notes (none) -> U4:VIN and CE to +3V3_CLEAN decoupling to GND
- C22: Notes (none) -> U1:GPIO0 to SW1 decouple to GND
- C23: value 1.0uF -> 1uF; Notes (none) -> U1:EN to SW2 decoupling to GND
- C3, C4: Notes (none) -> PS1:L1 to +3V3 decoupling to GND
- C5: Notes (none) -> +BATT to PS1:IN decoupling to GND
- C6: Notes (none) -> PS1: LX to PS1:BS
- C7: Notes PS1:FB series to +3V3 -> PS1:FB in series to +3V3
- C8, C9: Notes (none) -> R3 decoupling to +3V3_CLEAN
- D1: Notes (none) -> J2:VBUS to +BATT to avoid battery voltage flowing back into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
- FB1: Notes (none) -> PS1:FB to 3V3 clean
- FB2: Notes (none) -> +CAM_2V8 to J3:AVDD
- J1: Notes (none) -> Connector to 4 Wire Slip Ring Connector to Hull Board for I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
- J3: Notes (none) -> OV2640 24 pin camera connector
- J4, J5: Notes (none) -> 3mm IR LED connector
- J6: Notes (none) -> Connector for 6 × WS2812 RGB LED
- L1: Notes (none) -> PS1:LX to +3V3
- R1: Notes (none) -> J2:CC1 pull down
- R10: Notes (none) -> J3:RESETB pull up to +CAM_2V8
- R11: Notes (none) -> J3:XCLK series to GPIO15
- R12: Notes (none) -> J3:PWDN pull down
- R13: Notes (none) -> J3:SIO_C to GPIO5 pull up to +CAM_2V8
- R14: Notes (none) -> STATUS_LEDS to J6:Pin2 in series
- R15: Notes (none) -> U1:GPIO0 pull up to +3V3_CLEAN
- R16: Notes (none) -> U1:EN pull up to +3V3_CLEAN
- R2: Notes (none) -> J2:CC2 pull down
- R3: Notes (none) -> PS1:FB to +3v3 and FB1 in series
- R4: Notes (none) -> PS1:FB pull down
- R5: Notes (none) -> IR#1 to J4:Pin1 in series
- R6: Notes (none) -> IR#2 to J5:Pin1 in series
- R7: Notes (none) -> J3:SIO_D to GPIO4 pull up to +CAM_2V8
- R8: Notes (none) -> BUZZER to Q1:Base in series
- R9: Notes (none) -> R8 to Q1:Base pull down
- U1: Notes (none) -> ESP32 in tank turret
- U3: Notes (none) -> +3V3_CLEAN to +CAM2V8
- U4: Notes (none) -> +3V3_CLEAN to +CAM1V3
Changed lines of the file:
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@@
 			)
 		)
-		(property "Notes" ""
+		(property "Notes" "J3:RESETB pull up to +CAM_2V8"
 			(at 267.97 69.85 90)
 			(effects
@@
 			)
 		)
-		(property "Notes" ""
+		(property "Notes" "J3:SIO_C to GPIO5 pull up to +CAM_2V8"
 			(at 275.59 82.55 90)
 			(effects
@@
 			)
 		)
-		(property "Notes" ""
+		(property "Notes" "PS1:FB to +3v3 and FB1 in series"
 			(at 138.43 63.5 0)
 			(effects
@@
 			)
 		)
-		(property "Notes" ""
+		(property "Notes" "PS1:FB pull down"
 			(at 154.94 45.72 0)
 			(effects
@@
 			)
 		)
-		(property "Notes" ""
+		(property "Notes" "U4:VOUT to DVDD decoupling to GND"
 			(at 316.23 55.88 0)
 			(effects
@@
 			)
 		)
-		(property "Notes" ""
+		(property "Notes" "U3:VOUT to DOVDD decoupling to GND"
 			(at 311.15 33.02 0)
 			(effects
@@
 			)
 		)
-		(property "Notes" ""
+		(property "Notes" "J3:SIO_D to GPIO4 pull up to +CAM_2V8"
 			(at 246.38 101.6 90)
 			(effects
@@
 			)
 		)
-		(property "Notes" ""
+		(property "Notes" "J2:VBUS to +5V_USB decoupling to GND"
 			(at 67.31 243.84 0)
 			(effects
@@
 			)
 		)
-		(property "Notes" ""
+		(property "Notes" "PS1:L1 to +3V3 decoupling to GND"
 			(at 99.06 38.1 0)
 			(effects
@@
 			)
 		)
-		(property "Notes" ""
+		(property "Notes" "Connector for  6 × WS2812 RGB LED"
 			(at 374.65 162.56 0)
 			(effects
@@
 			)
 		)
-		(property "Notes" ""
+		(property "Notes" "AVDD decoupling to +CAM_AVDD_28"
 			(at 281.94 95.25 90)
 			(effects
@@
 			)
 		)
-		(property "Notes" ""
+		(property "Notes" "AVDD decoupling to +CAM_AVDD_28"
 			(at 294.64 95.25 90)
 			(effects
@@
 			)
 		)
-		(property "Notes" ""
+		(property "Notes" "J2:CC2 pull down"
 			(at 67.31 232.41 90)
 			(effects
@@
 			)
 		)
-		(property "Notes" ""
+		(property "Notes" "J2:VBUS to +5V_USB decoupling to GND"
 			(at 54.61 243.84 0)
 			(effects
@@
 			)
 		)
-		(property "Notes" ""
+		(property "Notes" "R3 decoupling to +3V3_CLEAN"
 			(at 181.61 66.04 0)
 			(effects
@@
 			)
 		)
-		(property "Notes" ""
+		(property "Notes" "PS1: LX to PS1:BS"
 			(at 124.46 30.48 90)
 			(effects
@@
 			)
 		)
-		(property "Notes" "PS1:FB series to +3V3"
+		(property "Notes" "PS1:FB in series to +3V3"
 			(at 130.81 63.5 90)
 			(effects
@@
 			)
 		)
-		(property "Notes" ""
+		(property "Notes" "PS1:LX to +3V3"
 			(at 106.68 44.45 90)
 			(effects
@@
 			)
 		)
-		(property "Notes" ""
+		(property "Notes" "J6:PIN1 to +3V3 decoupling to GND"
 			(at 347.98 153.67 0)
 			(effects
@@
 			)
 		)
-		(property "Notes" ""
+		(property "Notes" "3mm IR LED connector"
 			(at 259.08 222.25 0)
 			(effects
@@
 			)
 		)
-		(property "Notes" ""
+		(property "Notes" "R8 to Q1:Base pull down"
 			(at 257.81 171.45 0)
 			(effects
@@
 			)
 		)
-		(property "Notes" ""
+		(property "Notes" "3mm IR LED connector"
 			(at 259.08 209.55 0)
 			(effects
@@
 			)
 		)
-		(property "Notes" ""
+		(property "Notes" "R3 decoupling to +3V3_CLEAN"
 			(at 166.37 66.04 0)
 			(effects
@@
 			)
 		)
-		(property "Notes" ""
+		(property "Notes" "+3V3_CLEAN to +CAM2V8"
 			(at 346.71 34.29 0)
 			(effects
@@
 			)
 		)
-		(property "Notes" ""
+		(property "Notes" "U1:GPIO0 to SW1 decouple to GND"
 			(at 176.53 116.84 0)
 			(effects
@@
 			)
 		)
-		(property "Notes" ""
+		(property "Notes" "U3:VIN to +3V3_CLEAN decoupling to GND"
 			(at 383.54 33.02 0)
 			(effects
@@
 			)
 		)
-		(property "Notes" ""
+		(property "Notes" "J3:PWDN pull down"
 			(at 288.29 64.77 90)
 			(effects
@@
 			)
 		)
-		(property "Notes" ""
+		(property "Notes" "U3:VOUT to DOVDD decoupling to GND"
 			(at 299.72 33.02 0)
 			(effects
@@
 			)
 		)
-		(property "Notes" ""
+		(property "Notes" "J2:CC1 pull down"
 			(at 52.07 236.22 90)
 			(effects
@@
 			)
 		)
-		(property "Notes" ""
+		(property "Notes" "PS1:FB to 3V3 clean"
 			(at 156.21 62.23 90)
 			(effects
@@
 			)
 		)
-		(property "Notes" ""
+		(property "Notes" "+3V3_CLEAN to +CAM1V3"
 			(at 346.71 60.96 0)
 			(effects
@@
 			)
 		)
-		(property "Notes" ""
+		(property "Notes" "IR#1 to J4:Pin1 in series"
 			(at 243.84 209.55 90)
 			(effects
@@
 			)
 		)
-		(property "Notes" ""
+		(property "Notes" "U4:VIN and CE to +3V3_CLEAN decoupling to GND"
 			(at 381 59.69 0)
 			(effects
@@
 			)
 		)
-		(property "Notes" ""
+		(property "Notes" "J6:PIN1 to +3V3 decoupling to GND"
 			(at 361.95 153.67 0)
 			(effects
@@
 			)
 		)
-		(property "Notes" ""
+		(property "Notes" "U4:VOUT to DVDD decoupling to GND"
 			(at 300.99 55.88 0)
 			(effects
@@
 			)
 		)
-		(property "Notes" ""
+		(property "Notes" "J6:PIN1 to +3V3 decoupling to GND"
 			(at 335.28 153.67 0)
 			(effects
@@
 			)
 		)
-		(property "Notes" ""
+		(property "Notes" "J2:VBUS to +BATT to avoid battery voltage flowing back into USB"
 			(at 39.37 248.92 0)
 			(effects
@@
 			)
 		)
-		(property "Notes" ""
+		(property "Notes" "STATUS_LEDS to J6:Pin2 in series"
 			(at 349.25 168.91 90)
 			(effects
@@
 			)
 		)
-		(property "Notes" ""
+		(property "Notes" "PS1:L1 to +3V3 decoupling to GND"
 			(at 90.17 38.1 0)
 			(effects
@@
 			)
 		)
-		(property "Notes" ""
+		(property "Notes" "J3:XCLK series to GPIO15"
 			(at 264.16 52.07 90)
 			(effects
@@
 			)
 		)
-		(property "Notes" ""
+		(property "Notes" "U3:VOUT to DOVDD decoupling to GND"
 			(at 284.48 33.02 0)
 			(effects
@@
 			)
 		)
-		(property "Notes" ""
+		(property "Notes" "U4:VIN and CE to +3V3_CLEAN decoupling to GND"
 			(at 365.76 59.69 0)
 			(effects
@@
 			)
 		)
-		(property "Notes" ""
+		(property "Notes" "3V Piezo Buzzer"
 			(at 284.48 152.4 0)
 			(effects
@@
 			)
 		)
-		(property "Notes" ""
+		(property "Notes" "Connector to 4 Wire Slip Ring Connector to Hull Board for I2C and power"
 			(at 38.1 46.99 0)
 			(effects
@@
 			)
 		)
-		(property "Notes" ""
+		(property "Notes" "U1:EN pull up to +3V3_CLEAN"
 			(at 50.8 93.98 90)
 			(effects
@@
 			)
 		)
-		(property "Notes" ""
+		(property "Notes" "U3:VIN to +3V3_CLEAN decoupling to GND"
 			(at 368.3 33.02 0)
 			(effects
@@
 			)
 		)
-		(property "Notes" ""
+		(property "Notes" "IR#2 to J5:Pin1 in series"
 			(at 243.84 222.25 90)
 			(effects
@@
 			)
 		)
-		(property "Notes" ""
+		(property "Notes" "+CAM_2V8 to J3:AVDD"
 			(at 320.04 91.44 90)
 			(effects
@@
 			)
 		)
-		(property "Notes" ""
+		(property "Notes" "BUZZER to Q1:Base in series"
 			(at 250.19 163.83 90)
 			(effects
@@
 			)
 		)
-		(property "Notes" ""
+		(property "Notes" "ESP32 in tank turret"
 			(at 109.22 133.35 0)
 			(effects
@@
 			)
 		)
-		(property "Notes" ""
+		(property "Notes" "OV2640 24 pin camera connector"
 			(at 233.68 52.07 90)
 			(effects
@@
 			)
 		)
-		(property "Notes" ""
+		(property "Notes" "+BATT to PS1:IN decoupling to GND"
 			(at 99.06 57.15 0)
 			(effects
@@
 			)
 		)
-		(property "Notes" ""
+		(property "Notes" "U1:GPIO0 pull up to +3V3_CLEAN"
 			(at 180.34 93.98 90)
 			(effects
@@
 			)
 		)
-		(property "Value" "1.0uF"
+		(property "Value" "1uF"
 			(at 35.814 109.22 0)
 			(effects
@@
 			)
 		)
-		(property "Notes" ""
+		(property "Notes" "U1:EN to SW2 decoupling to GND"
 			(at 43.18 106.68 0)
 			(effects
