File: TankTurret/TankTurret.kicad_sch (KiCad schematic)
At the start: 59 parts, among them J1 Conn_01x04_Socket, J2 USB_C_Receptacle_USB2.0_16P, J3 Camera, J4 Conn_01x02, J5 Conn_01x02, J6 Conn_01x03, Q1 MMBT3904, SW1 SW_Push, SW2 SW_Push, U1 ESP32-S3-WROOM-1, U3 ME6211C28M5G, U4 LN1234B132MR-G

Commit message: Signed-off-by: SMAUG\Pete <pwbrophy@gmail.com>
Parts:
- removed J3: Camera, Jushuo:AFC07-S24ECA-00_flux, symbol Connector:Conn_01x24_Socket
- added C26: 100nF, Capacitor_SMD:C_0603_1608Metric, symbol Device:C
- added D2: PRTR5V0U2X, Package_TO_SOT_SMD:SOT-143, symbol Power_Protection:PRTR5V0U2X
- added D3: LED, LED_SMD:LED_0603_1608Metric, symbol Device:LED
- added D4: LED, LED_SMD:LED_0805_2012Metric, symbol Device:LED
- added FPC1: AFC07-S24ECA-00, EasyEDA2Kicad:FPC-SMD_AFC07-S24ECA-00, symbol Thundergeddon_custom:AFC07-S24ECA-00_OV2640
- added R17: 10k, Resistor_SMD:R_0603_1608Metric, symbol Device:R
- added R18: 1k, Resistor_SMD:R_0603_1608Metric, symbol Device:R
- C1: footprint Capacitor_SMD:C_0805_2012Metric -> Capacitor_SMD:C_0603_1608Metric; JLCPCB Part # (none) -> C14663
- C10, C11, C15, C17, C19, C22, C8: footprint Capacitor_SMD:C_0402_1005Metric -> Capacitor_SMD:C_0603_1608Metric; JLCPCB Part # (none) -> C14663
- C12, C14, C16, C20, C21, C9: footprint Capacitor_SMD:C_0201_0603Metric -> Capacitor_SMD:C_0603_1608Metric; JLCPCB Part # (none) -> C15849
- C13: footprint Capacitor_SMD:C_0201_0603Metric -> Capacitor_SMD:C_0805_2012Metric; JLCPCB Part # (none) -> C1779
- C2: JLCPCB Part # (none) -> C15850
- C23: JLCPCB Part # (none) -> C15849
- C25: JLCPCB Part # (none) -> C14663
- D1: JLCPCB Part # (none) -> C8598; Manufacturer_Name (none) -> Jiangsu Changjing; Manufacturer_Part_Number (none) -> B5819W SL
- FB1, FB2: JLCPCB Part # (none) -> C1002
- J1: symbol Connector:Conn_01x04_Socket -> Thundergeddon_Power:Turret_Slip_Ring_Connector; JLCPCB Part # C262643 -> (none); now not fitted
- J2: Notes (none) -> USB connector for power and uploading
- PS1: symbol SY8113BADC:SY8113BADC -> Thundergeddon_Power:SY8113BADC_Thundergeddon; Notes (none) -> 7.4V -> 3.3V Buck
- Q1: JLCPCB Part # (none) -> C20526; Manufacturer_Name (none) -> Jiangsu Changjing; Manufacturer_Part_Number (none) -> MMBT3904(RANGE:100-300); Notes (none) -> Buzzer Transistor
- R1, R2: footprint Resistor_SMD:R_0402_1005Metric -> Resistor_SMD:R_0603_1608Metric; JLCPCB Part # (none) -> C23186
- R10, R12, R15, R16: footprint Resistor_SMD:R_0402_1005Metric -> Resistor_SMD:R_0603_1608Metric; JLCPCB Part # (none) -> C25804
- R11: footprint Resistor_SMD:R_0402_1005Metric -> Resistor_SMD:R_0603_1608Metric; JLCPCB Part # (none) -> C23140
- R13, R7: footprint Resistor_SMD:R_0402_1005Metric -> Resistor_SMD:R_0603_1608Metric; JLCPCB Part # (none) -> C23162
- R14: footprint Resistor_SMD:R_0402_1005Metric -> Resistor_SMD:R_0603_1608Metric; JLCPCB Part # (none) -> C23138
- R5, R6: footprint Resistor_SMD:R_0402_1005Metric -> Resistor_SMD:R_0603_1608Metric; JLCPCB Part # (none) -> C22962
- R8: footprint Resistor_SMD:R_0402_1005Metric -> Resistor_SMD:R_0603_1608Metric; JLCPCB Part # (none) -> C21190
- SW1, SW2: JLCPCB Part # (none) -> C318884; Manufacturer_Name (none) -> XKB Connection; Manufacturer_Part_Number (none) -> TS-1187A-B-A-B; Notes (none) -> EN Switch
- U3: symbol EasyEDA2Kicad:ME6211C28M5G -> Thundergeddon_Power:ME6211C28M5G_Thundergeddon; JLCPCB Part # (none) -> C53099; Manufacturer_Name (none) -> MICRONE; Manufacturer_Part_Number (none) -> ME6211C28M5G-N
- U4: symbol EasyEDA2Kicad:LN1234B132MR-G -> Thundergeddon_Power:LN1234B132MR-G_Thundergeddon; JLCPCB Part # (none) -> C3008051; Manufacturer_Name (none) -> NATLINEAR; Manufacturer_Part_Number (none) -> LN1234B132MR-G
Connections:
- net +3V3: now also R15.1, R16.1, U1.2 (3V3), C26.2, D2.4 (VCC), R18.2
- net +3V3_CLEAN: no longer R15.1, R16.1, U1.2 (3V3)
- net +BATT: now also R17.2
- net +CAM_1V3: now also FPC1.10 (DVDD)
- net +CAM_2V8: now also FPC1.11 (DOVDD)
- net +CAM_AVDD_2V8: now also FPC1.4 (AVDD)
- net GND: now also C26.1, D2.1 (GND), D3.1 (K), FPC1.15 (DGND), FPC1.2 (AGND)
- net GPIO10: now also FPC1.20 (DATA5)
- net GPIO11: now also FPC1.19 (DATA2)
- net GPIO12: now also FPC1.18 (DATA6)
- net GPIO13: now also FPC1.17 (PCLK)
- net GPIO16: now also FPC1.12 (DATA9)
- net GPIO17: now also FPC1.14 (DATA8)
- net GPIO18: now also FPC1.16 (DATA7)
- net GPIO4: now also FPC1.3 (SIOD)
- net GPIO5: now also FPC1.5 (SIOC)
- net GPIO6: now also FPC1.7 (VSYNC)
- net GPIO7: now also FPC1.9 (HREF)
- net GPIO8: now also FPC1.22 (DATA4)
- net GPIO9: now also FPC1.21 (DATA3)
- net USB_D+: now also D2.3 (I/O2)
- net USB_D-: now also D2.2 (I/O1)
- net at R10.2: now also FPC1.6 (RESETB)
- net at R12.2: now also FPC1.8 (PWDN)
- net at R11.2: now also FPC1.13 (XCLK1)
- net GPIO48: now reaches U1.25 (GPIO48/SPICLK_N/SUBSPICLK_N_DIFF)
- net GPIO48: now also D4.1 (K)
- new net: D4.2 (A), R18.1
- new net: D3.2 (A), R17.1
- no-connect marks 5 -> 21
Other:
- note added: "GREEN GPIO"
- note added: "RED +BATT POWER"
- note added: "Turret: External WS2812 6 × RGB LED"
- moved on the sheet: C1, C10, C11, C12, C13, C14, C15, C16, C17, C19, C2, C20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
