File: TankTurret/TankTurret.kicad_sch (KiCad schematic)
At the start: 65 parts, among them J1 Conn_01x04_Socket, J2 USB_C_Receptacle_USB2.0_16P, J4 Conn_01x02, J5 Conn_01x02, J6 Conn_01x03, Q1 MMBT3904, SW1 SW_Push, SW2 SW_Push, U1 ESP32-S3-WROOM-1, U3 ME6211C28M5G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

Commit message: Signed-off-by: SMAUG\Pete <pwbrophy@gmail.com>
Parts:
- C10, C11, C17, C19: footprint Capacitor_SMD:C_0603_1608Metric -> Capacitor_SMD:C_0402_1005Metric; JLCPCB Part # C14663 -> C1525
- J2: footprint Connector_USB:USB_C_Receptacle_HRO_TYPE-C-31-M-12 -> EasyEDA2Kicad:USB-C_SMD-TYPE-C-31-M-12_1; symbol Connector:USB_C_Receptacle_USB2.0_16P -> EasyEDA2Kicad:TYPE-C-31-M-12; LCSC Part (none) -> C165948
Connections:
- net +5V_USB: now also J2.A4B9 (VBUS), J2.B4A9 (VBUS); no longer J2.A4 (VBUS), J2.A9 (VBUS), J2.B4 (VBUS), J2.B9 (VBUS)
- net GND: now also J2.1 (EH), J2.2 (EH), J2.3 (EH), J2.4 (EH), J2.A1B12 (GND), J2.B1A12 (GND); no longer J2.A1 (GND), J2.A12 (GND), J2.B1 (GND), J2.B12 (GND), J2.S1 (SHIELD)
- net GPIO10: now also FPC1.19 (DATA2); no longer FPC1.20 (DATA5)
- net GPIO11: now also FPC1.20 (DATA5); no longer FPC1.19 (DATA2)
- net GPIO12: now also FPC1.21 (DATA3); no longer FPC1.18 (DATA6)
- net GPIO13: now also FPC1.22 (DATA4); no longer FPC1.17 (PCLK)
- net GPIO15: now also FPC1.12 (DATA9); no longer R11.1
- net GPIO16: now also R11.1; no longer FPC1.12 (DATA9)
- net GPIO8: now also FPC1.17 (PCLK); no longer FPC1.22 (DATA4)
- net GPIO9: now also FPC1.18 (DATA6); no longer FPC1.21 (DATA3)
- net at J2.A5 (CC1): now also R2.1; no longer R1.1
- net at J2.B5 (CC2): now also R1.1; no longer R2.1
Other:
- moved on the sheet: C1, C2, D1, R1, R2

Commit message: Signed-off-by: SMAUG\Pete <pwbrophy@gmail.com>
Parts:
- removed BZ1: Buzzer, Buzzer_Beeper:Buzzer_12x9.5RM7.6, symbol Device:Buzzer
- added J3: Conn_01x02, Connector_PinHeader_2.54mm:PinHeader_1x02_P2.54mm_Vertical, symbol Connector_Generic:Conn_01x02
- added R19, R20: 4.7k, Resistor_SMD:R_0603_1608Metric, symbol Device:R
Connections:
- net +3V3: now also J3.1 (Pin_1), R19.1, R20.1
- net I2C SCL: now also R20.2
- net I2C SDA: now also R19.2
- net IR #1: now also U1.33 (MTDO/GPIO40/CLK_OUT2); no longer U1.32 (MTCK/GPIO39/CLK_OUT3/SUBSPICS1)
- net IR #2: now also U1.32 (MTCK/GPIO39/CLK_OUT3/SUBSPICS1); no longer U1.33 (MTDO/GPIO40/CLK_OUT2)
- net at Q1.3 (C): now also J3.2 (Pin_2)

Commit message: Signed-off-by: SMAUG\Pete <pwbrophy@gmail.com>
Parts:
- added TP1, TP10, TP11, TP12, TP13, TP14, TP15, TP16, TP2, TP3, TP4, TP5, TP6, TP7, TP8, TP9: TestPoint, TestPoint:TestPoint_Pad_D1.0mm, symbol Connector:TestPoint
Connections:
- net +3V3: now also TP1.1
- net +3V3_CLEAN: now also TP2.1
- net +5V_USB: now also TP7.1
- net +BATT: now also TP3.1
- net +CAM_1V3: now also TP5.1
- net +CAM_2V8: now also TP4.1
- net GND: now also TP6.1
- net I2C SCL: now also TP11.1
- net I2C SDA: now also TP12.1
- net USB_D+: now also TP8.1
- net USB_D-: now also TP9.1
- net at J6.2 (Pin_2), R14.1: now also TP16.1
- net at J3.2 (Pin_2), Q1.3 (C): now also TP13.1
- net at FPC1.13 (XCLK1), R11.2: now also TP10.1
- net at J5.1 (Pin_1), R6.1: now also TP15.1
- net at J4.1 (Pin_1), R5.1: now also TP14.1
Other:
- moved on the sheet: J1, J4, J5, J6, R11, R5, R6

Commit message: Signed-off-by: SMAUG\Pete <pwbrophy@gmail.com>
Parts:
- added C27: 100nF, Capacitor_SMD:C_0603_1608Metric, symbol Device:C
- added C28: 10uF, Capacitor_SMD:C_0805_2012Metric, symbol Device:C
Connections:
- net +3V3: now also C27.2, C28.2
- net GND: now also C27.1, C28.1
Other:
- moved on the sheet: C22, C23, R15, R16, R19, R20, SW1, SW2, U1

Commit message: Signed-off-by: SMAUG\Pete <pwbrophy@gmail.com>
Parts:
- FPC1: JLCPCB Part # (none) -> C262643
- R10: Notes J3:RESETB pull up to +CAM_2V8 -> FPC1:RESETB pull up to +CAM_2V8
- R11: Notes J3:XCLK series to GPIO15 -> FPC1:XCLK series to GPIO15
- R12: Notes J3:PWDN pull down -> FPC1:PWDN pull down
- TP1, TP10, TP11, TP12, TP13, TP14, TP15, TP16, TP2, TP3, TP4, TP5, TP6, TP7, TP8, TP9: now left out of the parts list
Changed lines of the file:
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@@
 	(wire
 		(pts
-			(xy 104.14 222.25) (xy 106.68 222.25)
+			(xy 101.6 222.25) (xy 106.68 222.25)
 		)
 		(stroke
@@
 	)
 	(label "+5V_USB"
-		(at 104.14 222.25 180)
+		(at 101.6 222.25 180)
 		(effects
 			(font
@@
 			)
 		)
-		(property "Notes" "J3:RESETB pull up to +CAM_2V8"
+		(property "Notes" "FPC1:RESETB pull up to +CAM_2V8"
 			(at 262.89 81.28 90)
 			(effects
@@
 		(unit 1)
 		(exclude_from_sim no)
-		(in_bom yes)
-		(on_board yes)
+		(in_bom no)
+		(on_board no)
 		(dnp no)
 		(property "Reference" "TP10"
@@
 		(unit 1)
 		(exclude_from_sim no)
-		(in_bom yes)
-		(on_board yes)
+		(in_bom no)
+		(on_board no)
 		(dnp no)
 		(property "Reference" "TP15"
@@
 		(unit 1)
 		(exclude_from_sim no)
-		(in_bom yes)
-		(on_board yes)
+		(in_bom no)
+		(on_board no)
 		(dnp no)
 		(property "Reference" "TP11"
@@
 		(unit 1)
 		(exclude_from_sim no)
-		(in_bom yes)
-		(on_board yes)
+		(in_bom no)
+		(on_board no)
 		(dnp no)
 		(fields_autoplaced yes)
@@
 		(unit 1)
 		(exclude_from_sim no)
-		(in_bom yes)
-		(on_board yes)
+		(in_bom no)
+		(on_board no)
 		(dnp no)
 		(fields_autoplaced yes)
@@
 		(unit 1)
 		(exclude_from_sim no)
-		(in_bom yes)
-		(on_board yes)
+		(in_bom no)
+		(on_board no)
 		(dnp no)
 		(fields_autoplaced yes)
@@
 			)
 		)
+		(property "JLCPCB Part #" "C262643"
+			(at 226.06 64.77 0)
+			(effects
+				(font
+					(size 1.27 1.27)
+				)
+				(hide yes)
+			)
+		)
 		(pin "9"
 		)
@@
 		(unit 1)
 		(exclude_from_sim no)
-		(in_bom yes)
-		(on_board yes)
+		(in_bom no)
+		(on_board no)
 		(dnp no)
 		(property "Reference" "TP14"
@@
 		(unit 1)
 		(exclude_from_sim no)
-		(in_bom yes)
-		(on_board yes)
+		(in_bom no)
+		(on_board no)
 		(dnp no)
 		(fields_autoplaced yes)
@@
 		(unit 1)
 		(exclude_from_sim no)
-		(in_bom yes)
-		(on_board yes)
+		(in_bom no)
+		(on_board no)
 		(dnp no)
 		(property "Reference" "TP12"
@@
 		(unit 1)
 		(exclude_from_sim no)
-		(in_bom yes)
-		(on_board yes)
+		(in_bom no)
+		(on_board no)
 		(dnp no)
 		(fields_autoplaced yes)
@@
 			)
 		)
-		(property "Notes" "J3:PWDN pull down"
+		(property "Notes" "FPC1:PWDN pull down"
 			(at 283.21 76.2 90)
 			(effects
@@
 		(unit 1)
 		(exclude_from_sim no)
-		(in_bom yes)
-		(on_board yes)
+		(in_bom no)
+		(on_board no)
 		(dnp no)
 		(fields_autoplaced yes)
@@
 		(unit 1)
 		(exclude_from_sim no)
-		(in_bom yes)
-		(on_board yes)
+		(in_bom no)
+		(on_board no)
 		(dnp no)
 		(fields_autoplaced yes)
@@
 		(unit 1)
 		(exclude_from_sim no)
-		(in_bom yes)
-		(on_board yes)
+		(in_bom no)
+		(on_board no)
 		(dnp no)
 		(property "Reference" "TP13"
@@
 			)
 		)
-		(property "Notes" "J3:XCLK series to GPIO15"
+		(property "Notes" "FPC1:XCLK series to GPIO15"
 			(at 265.43 54.61 90)
 			(effects
@@
 		(unit 1)
 		(exclude_from_sim no)
-		(in_bom yes)
-		(on_board yes)
+		(in_bom no)
+		(on_board no)
 		(dnp no)
 		(fields_autoplaced yes)
@@
 		(unit 1)
 		(exclude_from_sim no)
-		(in_bom yes)
-		(on_board yes)
+		(in_bom no)
+		(on_board no)
 		(dnp no)
 		(property "Reference" "TP16"
@@
 		(unit 1)
 		(exclude_from_sim no)
-		(in_bom yes)
-		(on_board yes)
+		(in_bom no)
+		(on_board no)
 		(dnp no)
 		(fields_autoplaced yes)

Commit message: Signed-off-by: SMAUG\Pete <pwbrophy@gmail.com>
Parts:
- added C29: 22uF, Capacitor_SMD:C_0805_2012Metric, symbol Device:C
- added R21, R22: 33Ω, Resistor_SMD:R_0402_1005Metric, symbol Device:R
Connections:
- net +3V3: now also C29.2
- net GND: now also C29.1
- net I2C SCL: now also R22.1; no longer TP11.1, U1.24 (GPIO47/SPICLK_P/SUBSPICLK_P_DIFF)
- net I2C SDA: now also R21.1; no longer TP12.1, U1.23 (GPIO21)
- new net: R21.2, TP11.1, U1.23 (GPIO21)
- new net: R22.2, TP12.1, U1.24 (GPIO47/SPICLK_P/SUBSPICLK_P_DIFF)
Other:
- moved on the sheet: C18, C24, C25, R19, R20, TP11, TP12

Commit message: Signed-off-by: SMAUG\Pete <pwbrophy@gmail.com>
Parts:
- removed TP9: TestPoint, TestPoint:TestPoint_Pad_D1.0mm, symbol Connector:TestPoint
- J1: JLCPCB Part # (none) -> C157925; now fitted
Connections:
- net +3V3: no longer C26.2, D2.4 (VCC)
- net +5V_USB: now also C26.2, D2.4 (VCC)
- net GND: now also TP8.1
- net USB_D+: no longer TP8.1
- net STATUS_LEDS renamed WS2812_LEDS

Commit message: Signed-off-by: SMAUG\Pete <pwbrophy@gmail.com>
Parts:
- removed C22: 100nF, Capacitor_SMD:C_0603_1608Metric, symbol Device:C
- added R23, R24: 22Ω, Resistor_SMD:R_0402_1005Metric, symbol Device:R
- added R25: 4.7k, Resistor_SMD:R_0603_1608Metric, symbol Device:R
- J1: value Conn_01x04_Socket -> Conn_01x05_Socket; footprint Connector_JST:JST_XH_S4B-XH-A_1x04_P2.50mm_Horizontal -> Connector_JST:JST_PH_S5B-PH-K_1x05_P2.00mm_Horizontal; symbol Thundergeddon_Power:Turret_Slip_Ring_Connector -> Connector:Conn_01x05_Socket; JLCPCB Part # C157925 -> C157923; Notes Connector to 4 Wire Slip Ring Connector to Hull Board for I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 -> Connector to 5 Wire Slip Ring Connector to Hull Board for I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
- R17: value 10k -> 2.2k; JLCPCB Part # C25804 -> C25879
Connections:
- net +3V3: now also R25.1
- net GND: now also J1.3 (Pin_3); no longer J1.2 (Pin_2)
- net I2C SCL: now also J1.5 (Pin_5); no longer J1.4 (Pin_4)
- net I2C SDA: now also J1.4 (Pin_4); no longer J1.3 (Pin_3)
- net USB_D+: now also R24.1; no longer U1.14 (GPIO20/U1CTS/ADC2_CH9/CLK_OUT1/USB_D+)
- net USB_D-: now also R23.2; no longer U1.13 (GPIO19/U1RTS/ADC2_CH8/CLK_OUT2/USB_D-)
- net INT: now reaches U1.22 (GPIO14/TOUCH14/ADC2_CH3/FSPIWP/FSPIDQS/SUBSPIWP)
- net INT: now also J1.2 (Pin_2), R25.2
- new net USB_D+_ESP32: R24.2, U1.14 (GPIO20/U1CTS/ADC2_CH9/CLK_OUT1/USB_D+)
- new net USB_D-_ESP32: R23.1, U1.13 (GPIO19/U1RTS/ADC2_CH8/CLK_OUT2/USB_D-)
- no-connect marks 21 -> 20
Other:
- note added: "Turret: Slip Ring Connector"
- note removed: "Turret: Slip Ring Connector and Expansion Connections"
- moved on the sheet: R2
