File: TankTurret/TankTurret.kicad_sch (KiCad schematic)
At the start: 89 parts, among them J1 Conn_01x05_Socket, J2 USB_C_Receptacle_USB2.0_16P, J3 Conn_01x02, J4 Conn_01x02, J5 Conn_01x02, J6 Conn_01x03, Q1 MMBT3904, SW1 SW_Push, SW2 SW_Push, U1 ESP32-S3-WROOM-1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

Commit message: V0.2 Files sent to JLC PCB on 15/03/2026
Parts:
- J3: now not fitted; now left out of the parts list
- J4, J5, J6: now left out of the parts list
- R11: Notes FPC1:XCLK series to GPIO15 -> FPC1:XCLK series to GPIO16
- R17: JLCPCB Part # C25879 -> C4190
- R21: JLCPCB Part # C23140 -> C25105; Notes FPC1:XCLK series to GPIO15 -> Series Resistor SDA
- R22: JLCPCB Part # C23140 -> C25105; Notes FPC1:XCLK series to GPIO15 -> Series Resistor SCL
Changed lines of the file:
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@@
 	(wire
 		(pts
+			(xy 101.6 237.49) (xy 106.68 237.49)
+		)
+		(stroke
+			(width 0)
+			(type default)
+		)
+	)
+	(wire
+		(pts
 			(xy 297.18 102.87) (xy 303.53 102.87)
 		)
@@
 	(wire
 		(pts
+			(xy 101.6 234.95) (xy 106.68 234.95)
+		)
+		(stroke
+			(width 0)
+			(type default)
+		)
+	)
+	(wire
+		(pts
 			(xy 128.27 30.48) (xy 135.89 30.48)
 		)
@@
 	)
 	(label "USB_D-"
-		(at 105.41 229.87 180)
+		(at 101.6 229.87 180)
 		(effects
 			(font
@@
 	)
 	(label "USB_D+"
-		(at 105.41 232.41 180)
+		(at 101.6 232.41 180)
 		(effects
 			(font
@@
 	)
 	(label "USB_D+"
-		(at 106.68 237.49 180)
+		(at 101.6 237.49 180)
 		(effects
 			(font
@@
 	)
 	(label "USB_D-"
-		(at 106.68 234.95 180)
+		(at 101.6 234.95 180)
 		(effects
 			(font
@@
 			)
 		)
-		(property "JLCPCB Part #" "C23140"
+		(property "JLCPCB Part #" "C25105"
 			(at 197.358 194.818 0)
 			(effects
@@
 			)
 		)
-		(property "Notes" "FPC1:XCLK series to GPIO15"
+		(property "Notes" "Series Resistor SCL"
 			(at 176.53 170.18 90)
 			(effects
@@
 		(unit 1)
 		(exclude_from_sim no)
-		(in_bom yes)
+		(in_bom no)
 		(on_board yes)
 		(dnp yes)
@@
 		(unit 1)
 		(exclude_from_sim no)
-		(in_bom yes)
+		(in_bom no)
 		(on_board yes)
-		(dnp no)
+		(dnp yes)
 		(fields_autoplaced yes)
 		(property "Reference" "J3"
@@
 		(unit 1)
 		(exclude_from_sim no)
-		(in_bom yes)
+		(in_bom no)
 		(on_board yes)
 		(dnp yes)
@@
 		(unit 1)
 		(exclude_from_sim no)
-		(in_bom yes)
+		(in_bom no)
 		(on_board yes)
 		(dnp yes)
@@
 			)
 		)
-		(property "JLCPCB Part #" "C25879"
+		(property "JLCPCB Part #" "C4190"
 			(at 370.078 237.998 0)
 			(effects
@@
 		(dnp no)
 		(property "Reference" "R23"
-			(at 84.328 227.838 90)
+			(at 83.058 227.838 90)
 			(effects
 				(font
@@
 			)
 		)
-		(property "Notes" "FPC1:XCLK series to GPIO15"
+		(property "Notes" "FPC1:XCLK series to GPIO16"
 			(at 265.43 54.61 90)
 			(effects
@@
 			)
 		)
-		(property "JLCPCB Part #" "C23140"
+		(property "JLCPCB Part #" "C25105"
 			(at 197.358 184.658 0)
 			(effects
@@
 			)
 		)
-		(property "Notes" "FPC1:XCLK series to GPIO15"
+		(property "Notes" "Series Resistor SDA"
 			(at 176.53 160.02 90)
 			(effects
