File: TankHull/TankHull.kicad_pcb (KiCad board)
At the start: 2 copper layers, 77.9 x 40.6 mm, 65 parts, among them J1 SlipRing_4, J2 Conn_01x02_Socket, J3 Conn_01x02_Socket, J4 Conn_01x02_Socket, J5 Conn_01x02_Socket, J7 Conn_01x05, Q1 Q_PMOS, U10 TSSP77038TR, U11 TSSP77038TR, U12 TSSP77038TR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

Commit message: tweaks
Parts:
- removed IR N TST: TestPoint_Pad_D1.0mm, TestPoint:TestPoint_Pad_D1.0mm
- removed LM1 TST: TestPoint_Pad_D1.0mm, TestPoint:TestPoint_Pad_D1.0mm
- removed LM2 TST: TestPoint_Pad_D1.0mm, TestPoint:TestPoint_Pad_D1.0mm
- removed MS TST: TestPoint_Pad_D1.0mm, TestPoint:TestPoint_Pad_D1.0mm
- removed TP1: TestPoint, TestPoint:TestPoint_Pad_D1.0mm
- added C2: 4.7uF, Capacitor_SMD:C_0805_2012Metric, B.Cu at (151.8, 100.1)
- added R1: 47, Resistor_SMD:R_0603_1608Metric, B.Cu at (150.4, 103.4)
- added TP3: TestPoint, TestPoint:TestPoint_Pad_D1.0mm, B.Cu at (102.9, 108.6)
- added TP4: TestPoint, TestPoint:TestPoint_Pad_D1.0mm, B.Cu at (102.9, 106.5)
- added TP5: TestPoint, TestPoint:TestPoint_Pad_D1.0mm, B.Cu at (102.9, 104.4)
- added TP8: TestPoint, TestPoint:TestPoint_Pad_D1.0mm, B.Cu at (102.9, 102.3)
- U10, U11, U12, U4, U5, U6, U7, U9: value TSSP77038TR -> IRM-V838M3-C/TR1; footprint Vishay IR receiver:TSSP77038TR_VIS -> Everlight IR receiver:XDCR_IRM-V838M3_TR1
- moved C23 3.60 mm to (86.9, 117.2), turned to 135 degrees
- moved C22 2.67 mm to (85.0, 103.8), turned to 180 degrees
- moved C20 2.38 mm to (85.7, 90.4), turned to 135 degrees
- moved C18 1.79 mm to (149.5, 89.4)
- moved J5 1.69 mm to (90.7, 115.2)
- moved C25 1.53 mm to (150.4, 115.0)
- moved C24 1.42 mm to (119.2, 117.9)
- moved C16 1.20 mm to (152.0, 103.8)
- moved C19 0.94 mm to (117.5, 87.4)
- moved J7 0.90 mm to (132.6, 117.4)
- turned U10 to 135 degrees
- turned U11 to 180 degrees
- turned U12 to -135 degrees
- turned U4 to -90 degrees
- turned U5 to -45 degrees
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Connections:
- C16 pad 2: +3V3_HULL -> Net-(U4-VCC)
- U10 pad 4: (no net) -> GND
- U11 pad 4: (no net) -> GND
- U12 pad 4: (no net) -> GND
- U4 pad 2: +3V3_HULL -> Net-(U4-VCC)
- U4 pad 4: (no net) -> GND
- U5 pad 4: (no net) -> GND
- U6 pad 4: (no net) -> GND
- U7 pad 4: (no net) -> GND
- U9 pad 4: (no net) -> GND
Routing:
- net Net-(U4-VCC): track 0.00 -> 8.83 mm
- net +3V3_HULL: track 247.6 -> 239.9 mm
- net /IR Receive W: track 63.7 -> 60.6 mm
- net /IR Receive NW: track 95.9 -> 93.1 mm
- net /Left Drive Motor 1: track 11.2 -> 9.14 mm
- net /IR Receive NE: track 94.0 -> 96.0 mm
- net +BATT: track 120.2 -> 118.4 mm
- net /Left Drive Motor 2: track 11.1 -> 9.42 mm
- net /IR Receive SE: track 28.8 -> 30.3 mm
- net /IR Receive N: track 108.0 -> 109.1 mm
- net /Motors Sleep: track 42.0 -> 41.1 mm
- net /Left Motor Control 1: track 10.9 -> 10.1 mm
- net /IR Receive E: track 62.2 -> 62.9 mm
- net /IR Receive SW: track 31.1 -> 30.6 mm
- net GND: track 48.5 -> 48.0 mm
Other:
- board text added: "L DRV 1"
- board text added: "L DRV 2"
- board text added: "TEST"
- board text removed: "BAT TEST"
- board text removed: "LD1 TST"
- board text removed: "LD2 TST"

Commit message: camera connector
Parts:
- added C17: 4.7uF, Capacitor_SMD:C_0805_2012Metric, B.Cu at (148.2, 88.5)
- added C26: 4.7uF, Capacitor_SMD:C_0805_2012Metric, B.Cu at (119.5, 87.6)
- added C27: 4.7uF, Capacitor_SMD:C_0805_2012Metric, B.Cu at (151.9, 114.3)
- added C28: 4.7uF, Capacitor_SMD:C_0805_2012Metric, B.Cu at (116.8, 117.7)
- added C29: 4.7uF, Capacitor_SMD:C_0805_2012Metric, B.Cu at (87.9, 117.9)
- added C30: 4.7uF, Capacitor_SMD:C_0805_2012Metric, B.Cu at (84.8, 100.9)
- added C31: 4.7uF, Capacitor_SMD:C_0805_2012Metric, B.Cu at (87.3, 88.2)
- added R12: 47Ω, Resistor_SMD:R_0603_1608Metric, B.Cu at (120.0, 116.4)
- added R2: 47Ω, Resistor_SMD:R_0603_1608Metric, B.Cu at (149.6, 90.7)
- added R20: 47Ω, Resistor_SMD:R_0603_1608Metric, B.Cu at (86.6, 114.8)
- added R21: 47Ω, Resistor_SMD:R_0603_1608Metric, B.Cu at (86.5, 103.5)
- added R22: 47Ω, Resistor_SMD:R_0603_1608Metric, B.Cu at (83.7, 91.5)
- added R5: 47Ω, Resistor_SMD:R_0603_1608Metric, B.Cu at (116.2, 89.0)
- added R6: 47Ω, Resistor_SMD:R_0603_1608Metric, B.Cu at (148.7, 115.7)
- R1: value 47 -> 47Ω
- moved C20 69.1 mm to (149.5, 117.1), turned to 45 degrees
- moved C25 69.1 mm to (85.8, 90.4), turned to 135 degrees
- moved C22 38.1 mm to (120.3, 118.0)
- moved C24 37.3 mm to (84.2, 104.9), turned to 90 degrees
- moved C23 2.39 mm to (85.2, 115.6), turned to -45 degrees
- moved C18 1.67 mm to (151.1, 90.0), turned to 135 degrees
- moved C19 1.56 mm to (115.9, 87.4), turned to 0 degrees
Connections:
- C18 pad 2: +3V3_HULL -> Net-(U5-VCC)
- C19 pad 2: +3V3_HULL -> Net-(U6-VCC)
- C20 pad 2: +3V3_HULL -> Net-(U12-VCC)
- C22 pad 2: +3V3_HULL -> Net-(U11-VCC)
- C23 pad 2: +3V3_HULL -> Net-(U10-VCC)
- C24 pad 2: +3V3_HULL -> Net-(U9-VCC)
- C25 pad 2: +3V3_HULL -> Net-(U7-VCC)
- U10 pad 2: +3V3_HULL -> Net-(U10-VCC)
- U11 pad 2: +3V3_HULL -> Net-(U11-VCC)
- U12 pad 2: +3V3_HULL -> Net-(U12-VCC)
- U5 pad 2: +3V3_HULL -> Net-(U5-VCC)
- U6 pad 2: +3V3_HULL -> Net-(U6-VCC)
- U7 pad 2: +3V3_HULL -> Net-(U7-VCC)
- U9 pad 2: +3V3_HULL -> Net-(U9-VCC)
Routing:
- net +3V3_HULL: track 239.9 -> 217.0 mm, vias 17 -> 18
- net Net-(U9-VCC): track 0.00 -> 8.11 mm
- net Net-(U12-VCC): track 0.00 -> 7.88 mm
- net Net-(U5-VCC): track 0.00 -> 7.84 mm
- net Net-(U6-VCC): track 0.00 -> 7.77 mm
- net Net-(U10-VCC): track 0.00 -> 7.70 mm
- net Net-(U11-VCC): track 0.00 -> 7.67 mm
- net Net-(U7-VCC): track 0.00 -> 7.04 mm
- net /IR Receive SW: track 30.6 -> 32.1 mm
- net /Motors Sleep: track 41.1 -> 40.6 mm
- net /IR Receive S: track 19.6 -> 20.1 mm

Commit message: Signed-off-by: SMAUG\Pete <pwbrophy@gmail.com>
Parts:
- removed R3, R7: 3.3kΩ, Resistor_SMD:R_0603_1608Metric
Connections:
- C29 pad 1: GND -> unconnected-(C29-Pad1)
- C31 pad 1: GND -> unconnected-(C31-Pad1)
- J1 pad 3: /SDA -> +3V3_HULL
- J1 pad 4: /SCL -> +3V3_HULL
- J7 pad 1: /SCL -> +3V3_HULL
- J7 pad 2: /SDA -> +3V3_HULL
- U8 pad 22: /SCL -> +3V3_HULL
- U8 pad 23: /SDA -> +3V3_HULL
Routing:
- net +3V3_HULL: track 217.0 -> 300.2 mm, vias 18 -> 22
- net /SDA: track 39.8 -> 0.00 mm, vias 2 -> 0
- net /SCL: track 37.2 -> 0.00 mm, vias 2 -> 0

Commit message: Signed-off-by: SMAUG\Pete <pwbrophy@gmail.com>
Parts:
- D9: footprint LED_SMD:LED_Kingbright_APA1606_1.6x0.6mm_Horizontal -> Diode_SMD:D_0603_1608Metric
- R10, R11, R13, R14, R18, R19, R8, R9: footprint Resistor_SMD:R_01005_0402Metric -> Resistor_SMD:R_0603_1608Metric
- moved R11 2.95 mm to (97.3, 109.4), turned to -90 degrees
- moved R9 2.77 mm to (97.5, 99.5), turned to -90 degrees
- moved C11 2.58 mm to (104.8, 114.9)
- moved R10 2.55 mm to (99.0, 109.4), turned to -90 degrees
- moved R8 2.47 mm to (99.0, 99.5), turned to -90 degrees
- moved C4 2.12 mm to (102.8, 90.7)
- moved C5 1.70 mm to (104.8, 90.7)
- moved R13 1.58 mm to (96.4, 102.0)
- moved R18 1.56 mm to (96.4, 106.7)
- moved C12 1.33 mm to (106.7, 115.0)
- moved C17 1.26 mm to (148.1, 87.2), turned to -45 degrees
- moved R14 1.19 mm to (96.4, 103.6)
- moved R19 1.17 mm to (96.4, 105.1)
- moved C27 1.05 mm to (150.8, 114.2), turned to -45 degrees
- moved J1 0.40 mm to (120.0, 112.2)
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Connections:
- C29 pad 1: unconnected-(C29-Pad1) -> GND
- C31 pad 1: unconnected-(C31-Pad1) -> GND
- J1 pad 3: +3V3_HULL -> /SDA
- J1 pad 4: +3V3_HULL -> /SCL
- J7 pad 1: +3V3_HULL -> /SCL
- J7 pad 2: +3V3_HULL -> /SDA
- U8 pad 22: +3V3_HULL -> /SCL
- U8 pad 23: +3V3_HULL -> /SDA
Routing:
- net +3V3_HULL: track 300.2 -> 233.5 mm, vias 22 -> 18
- net /SDA: track 0.00 -> 39.2 mm, vias 0 -> 2
- net /SCL: track 0.00 -> 37.0 mm, vias 0 -> 2
- net GND: track 48.0 -> 50.4 mm
- net /IR Receive W: track 60.4 -> 62.6 mm
- net /IR Receive NE: track 96.0 -> 97.6 mm
- net /IR Receive E: track 62.9 -> 64.0 mm
- net /IR Receive SW: track 32.1 -> 33.0 mm
- net /IR Receive SE: track 30.2 -> 30.9 mm
- net /IR Receive S: track 20.1 -> 20.8 mm
- net +BATT: track 118.4 -> 119.1 mm
- net /IR Receive NW: track 93.5 -> 94.1 mm
Other:
- board text added: "IR N"
- board text added: "L CTRL 1"
- board text added: "L CTRL 2"
- board text added: "SLEEP"
- board text removed: "TEST"
