File: TankHull/TankHull.kicad_pcb (KiCad board)
At the start: 2 copper layers, 77.9 x 40.6 mm, 78 parts, among them J1 SlipRing_4, J2 Conn_01x02_Socket, J3 Conn_01x02_Socket, J4 Conn_01x02_Socket, J5 Conn_01x02_Socket, J7 Conn_01x05, Q1 Q_PMOS, U10 IRM-V838M3-C/TR1, U11 IRM-V838M3-C/TR1, U12 IRM-V838M3-C/TR1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

Commit message: Signed-off-by: SMAUG\Pete <pwbrophy@gmail.com>
Parts:
- added REF**: MountingHole_2.2mm_M2, MountingHole:MountingHole_2.2mm_M2, B.Cu at (143.3, 86.0)
- added REF**: MountingHole_2.2mm_M2, MountingHole:MountingHole_2.2mm_M2, B.Cu at (94.8, 119.3)
- added REF**: MountingHole_2.2mm_M2, MountingHole:MountingHole_2.2mm_M2, B.Cu at (143.3, 119.3)
- added REF**: MountingHole_2.2mm_M2, MountingHole:MountingHole_2.2mm_M2, B.Cu at (94.8, 86.0)
- moved J7 1.95 mm to (132.6, 115.7)
- moved J4 1.90 mm to (87.0, 107.9)
- moved R17 1.05 mm to (140.2, 111.7)
- moved R4 0.62 mm to (142.1, 95.3)
- moved C11 0.60 mm to (104.8, 114.3)
- moved C12 0.60 mm to (106.7, 114.4)
- moved C6 0.60 mm to (106.0, 116.9)
- moved U3 0.60 mm to (99.9, 114.5)
- moved C8 0.60 mm to (105.4, 111.9)
- moved J5 0.35 mm to (90.6, 114.9)
- moved TP6 0.05 mm to (94.5, 115.0), turned to 180 degrees
- turned TP7 to 180 degrees
Routing:
- net +3V3_HULL: track 233.5 -> 206.3 mm, vias 18 -> 16
- net /IR Receive SW: track 33.0 -> 35.7 mm
- net /IR Receive NW: track 94.1 -> 96.7 mm
- net /IR Receive W: track 62.6 -> 64.8 mm
- net /IR Receive NE: track 97.6 -> 99.5 mm
- net /Turret Motor 1: track 11.3 -> 12.7 mm
- net /Turret Motor 2: track 12.1 -> 13.5 mm
- net /IR Receive N: track 109.5 -> 110.5 mm
- net /SDA: track 39.2 -> 38.4 mm
- net /Motors Sleep: track 40.6 -> 41.3 mm
- net /Turret Motor Control 2: track 16.8 -> 16.2 mm
- net /Turret Motor Control 1: track 15.9 -> 15.3 mm
- net /Left Motor Control 2: track 12.8 -> 12.2 mm
- net /Left Motor Control 1: track 10.1 -> 9.52 mm
- net Net-(Q1-G): track 2.14 -> 1.54 mm
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
Commit message: Signed-off-by: SMAUG\Pete <pwbrophy@gmail.com>
Parts:
- added D4: LED, LED_SMD:LED_0805_2012Metric, B.Cu at (108.0, 97.7)
- added R23: 10kΩ, Resistor_SMD:R_0603_1608Metric, B.Cu at (105.0, 118.3)
- added R24: 10kΩ, Resistor_SMD:R_0603_1608Metric, F.Cu at (105.8, 111.2)
- added R25: 10kΩ, Resistor_SMD:R_0603_1608Metric, F.Cu at (104.1, 94.8)
- added R26: 10kΩ, Resistor_SMD:R_0603_1608Metric, F.Cu at (99.0, 94.9)
- added R27: 10kΩ, Resistor_SMD:R_0603_1608Metric, F.Cu at (97.9, 97.0)
- added R28: 220, Resistor_SMD:R_0603_1608Metric, B.Cu at (107.2, 100.2)
- added R3: 10kΩ, Resistor_SMD:R_0603_1608Metric, F.Cu at (101.0, 110.8)
- added R7: 10kΩ, Resistor_SMD:R_0603_1608Metric, B.Cu at (106.2, 116.8)
- moved C8 2.71 mm to (108.0, 111.2), turned to -90 degrees
- moved TP6 2.60 mm to (97.2, 115.0)
- moved TP7 2.60 mm to (97.2, 112.6)
Connections:
- U2 pad 15: unconnected-(U2-AIN2-Pad15) -> GND
- U2 pad 16: unconnected-(U2-AIN1-Pad16) -> GND
- U3 pad 10: /Turret Motor Control 2 -> /Left Motor Control 2
- U3 pad 15: /Left Motor Control 2 -> /Turret Motor Control 2
- U3 pad 16: /Left Motor Control 1 -> /Turret Motor Control 1
- U3 pad 9: /Turret Motor Control 1 -> /Left Motor Control 1
- U8 pad 13: /Left Motor Control 1 -> /Turret Motor Control 1
- U8 pad 14: /Left Motor Control 2 -> /Turret Motor Control 2
- U8 pad 15: /Turret Motor Control 1 -> /Left Motor Control 1
- U8 pad 16: /Turret Motor Control 2 -> /Left Motor Control 2
- U8 pad 20: unconnected-(U8-IO1_7-Pad20) -> Net-(U8-IO1_7)
Routing:
- net GND: track 50.3 -> 62.9 mm, vias 14 -> 20
- net /Left Motor Control 1: track 9.52 -> 21.1 mm, vias 1 -> 3
- net /Left Motor Control 2: track 12.2 -> 20.7 mm, vias 1 -> 3
- net /Turret Motor Control 1: track 15.4 -> 7.94 mm, vias 2 -> 0
- net /Turret Motor Control 2: track 16.2 -> 11.4 mm, vias 2 -> 0
- net Net-(U8-IO1_7): track 0.00 -> 2.94 mm, vias 0 -> 1
- net /Left Drive Motor 1: track 8.78 -> 11.7 mm
- net Net-(U3-VINT): track 2.94 -> 5.87 mm
- net /Left Drive Motor 2: track 9.20 -> 11.7 mm
- net /Motors Sleep: track 41.3 -> 43.1 mm
- net /Right Motor Control 2: track 13.3 -> 15.1 mm
- net Net-(D4-A): track 0.00 -> 1.78 mm
- net /Right Motor Control 1: track 13.7 -> 15.2 mm

Commit message: Signed-off-by: SMAUG\Pete <pwbrophy@gmail.com>
Parts:
- removed Q1: Q_PMOS, Package_TO_SOT_SMD:SOT-23-3
- added Q2: AO3401A, EasyEDA2Kicad:SOT-23_L2.9-W1.3-P1.90-LS2.4-BR, F.Cu at (141.0, 91.0)
- added TP1: TestPoint, TestPoint:TestPoint_Pad_D1.0mm, B.Cu at (102.9, 100.3)
- J1: footprint Connector_JST:JST_XH_B4B-XH-A_1x04_P2.50mm_Vertical -> Connector_JST:JST_PH_B5B-PH-K_1x05_P2.00mm_Vertical
- moved R4 7.84 mm to (139.0, 88.1), turned to 180 degrees
- moved TP7 2.50 mm to (94.9, 113.6)
- moved TP6 2.37 mm to (94.9, 115.7)
Connections:
- J1 pad 3: /SDA -> /INT
- J1 pad 4: /SCL -> /SDA
- U8 pad 1: unconnected-(U8-~{INT}-Pad1) -> /INT
Routing:
- net /INT: track 0.00 -> 23.6 mm, vias 0 -> 2
- net /Left Drive Motor 1: track 11.7 -> 8.78 mm
- net /Left Drive Motor 2: track 11.7 -> 8.91 mm
- net +BATT: track 118.9 -> 120.2 mm, vias 5 -> 3
- net /VBAT_RAW: track 13.5 -> 12.6 mm, vias 7 -> 11
- net +3V3_HULL: track 206.3 -> 205.7 mm
- net GND: track 62.9 -> 63.4 mm
Other:
- board text added: "- +"
- board text added: "INT"
- board text added: "IO1_7"
- board text removed: "+"
- board text removed: "-"

Commit message: V0.2 Files sent to JLC PCB on 15/03/2026
Parts:
- R28: value 220 -> 220Ω
Routing:
- net GND: track 63.4 -> 61.6 mm
