File: TankHull/TankHull.kicad_sch (KiCad schematic)
At the start: 80 parts, among them J1 SlipRing_4, J2 Conn_01x02_Socket, J3 Conn_01x02_Socket, J4 Conn_01x02_Socket, J5 Conn_01x02_Socket, J7 Conn_01x05, Q1 Q_PMOS, U10 IRM-V838M3-C/TR1, U11 IRM-V838M3-C/TR1, U12 IRM-V838M3-C/TR1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

Commit message: Signed-off-by: SMAUG\Pete <pwbrophy@gmail.com>
Parts:
- removed R3, R7: 3.3kΩ, Resistor_SMD:R_0603_1608Metric, symbol Device:R
Connections:
- net SCL is gone; now on net +3V3_HULL: J1.4 (Pin_4), J7.1 (Pin_1), U8.22 (SCL)
- net SDA is gone; now on net +3V3_HULL: J1.3 (Pin_3), J7.2 (Pin_2), U8.23 (SDA)
Changed lines of the file:
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@@
 	(wire
 		(pts
-			(xy 55.88 109.22) (xy 55.88 115.57)
+			(xy 55.88 109.22) (xy 55.88 125.73)
 		)
 		(stroke
@@
 	(wire
 		(pts
-			(xy 66.04 109.22) (xy 66.04 111.76)
+			(xy 66.04 109.22) (xy 66.04 123.19)
 		)
 		(stroke
@@
 	(wire
 		(pts
-			(xy 55.88 123.19) (xy 55.88 125.73)
-		)
-		(stroke
-			(width 0)
-			(type default)
-		)
-	)
-	(wire
-		(pts
 			(xy 323.85 127) (xy 323.85 144.78)
 		)
@@
 	(wire
 		(pts
-			(xy 66.04 123.19) (xy 66.04 119.38)
-		)
-		(stroke
-			(width 0)
-			(type default)
-		)
-	)
-	(wire
-		(pts
 			(xy 176.53 115.57) (xy 176.53 120.65)
 		)
@@
 	)
 	(symbol
-		(lib_id "Device:R")
-		(at 55.88 119.38 0)
-		(unit 1)
-		(exclude_from_sim no)
-		(in_bom yes)
-		(on_board yes)
-		(dnp no)
-		(property "Reference" "R3"
-			(at 50.038 118.11 0)
-			(effects
-				(font
-					(size 1.27 1.27)
-				)
-				(justify left)
-			)
-		)
-		(property "Value" "3.3kΩ"
-			(at 48.26 120.396 0)
-			(effects
-				(font
-					(size 1.27 1.27)
-				)
-				(justify left)
-			)
-		)
-		(property "Footprint" "Resistor_SMD:R_0603_1608Metric"
-			(at 54.102 119.38 90)
-			(effects
-				(font
-					(size 1.27 1.27)
-				)
-				(hide yes)
-			)
-		)
-		(property "Datasheet" "~"
-			(at 55.88 119.38 0)
-			(effects
-				(font
-					(size 1.27 1.27)
-				)
-				(hide yes)
-			)
-		)
-		(property "Description" "100mW Thick Film Resistors 75V ±100ppm/℃ ±1% 3.3kΩ 0603 Chip Resistor - Surface Mount ROHS"
-			(at 55.88 119.38 0)
-			(effects
-				(font
-					(size 1.27 1.27)
-				)
-				(hide yes)
-			)
-		)
-		(property "JLCPCB Part #" "C22978"
-			(at 133.35 106.426 0)
-			(effects
-				(font
-					(size 1.27 1.27)
-				)
-				(hide yes)
-			)
-		)
-		(property "MANUFACTURER" "UNI-ROYAL"
-			(at 133.35 106.426 0)
-			(effects
-				(font
-					(size 1.27 1.27)
-				)
-				(hide yes)
-			)
-		)
-		(property "Manufacturer_Part_Number" "0603WAF3301T5E"
-			(at 133.35 106.426 0)
-			(effects
-				(font
-					(size 1.27 1.27)
-				)
-				(hide yes)
-			)
-		)
-		(pin "1"
-		)
-		(pin "2"
-		)
-		(instances
-			(project "TankHull"
-				(path "/39d4946a-74a0-412b-8dfb-423b23371da5"
-					(reference "R3")
-					(unit 1)
-				)
-			)
-		)
-	)
-	(symbol
 		(lib_id "power:GND")
 		(at 162.56 74.93 0)
@@
 					(unit 1)
 				)
-			)
-		)
-	)
-	(symbol
-		(lib_id "Device:R")
-		(at 66.04 115.57 0)
-		(unit 1)
-		(exclude_from_sim no)
-		(in_bom yes)
-		(on_board yes)
-		(dnp no)
-		(property "Reference" "R7"
-			(at 68.072 114.3 0)
-			(effects
-				(font
-					(size 1.27 1.27)
-				)
-				(justify left)
-			)
-		)
-		(property "Value" "3.3kΩ"
-			(at 68.072 116.84 0)
-			(effects
-				(font
-					(size 1.27 1.27)
-				)
-				(justify left)
-			)
-		)
-		(property "Footprint" "Resistor_SMD:R_0603_1608Metric"
-			(at 64.262 115.57 90)
-			(effects
-				(font
-					(size 1.27 1.27)
-				)
-				(hide yes)
-			)
-		)
-		(property "Datasheet" "~"
-			(at 66.04 115.57 0)
-			(effects
-				(font
-					(size 1.27 1.27)
-				)
-				(hide yes)
-			)
-		)
-		(property "Description" "100mW Thick Film Resistors 75V ±100ppm/℃ ±1% 3.3kΩ 0603 Chip Resistor - Surface Mount ROHS"
-			(at 66.04 115.57 0)
-			(effects
-				(font
-					(size 1.27 1.27)
-				)
-				(hide yes)
-			)
-		)
-		(property "JLCPCB Part #" "C22978"
-			(at 130.302 107.188 0)
-			(effects
-				(font
-					(size 1.27 1.27)
-				)
-				(hide yes)
-			)
-		)
-		(property "MANUFACTURER" "UNI-ROYAL"
-			(at 130.302 107.188 0)
-			(effects
-				(font
-					(size 1.27 1.27)
-				)
-				(hide yes)
-			)
-		)
-		(property "Manufacturer_Part_Number" "0603WAF3301T5E"
-			(at 129.286 108.458 0)
-			(effects
-				(font
-					(size 1.27 1.27)
-				)
-				(hide yes)
-			)
-		)
-		(pin "1"
-		)
-		(pin "2"
-		)
-		(instances
-			(project "TankHull"
-				(path "/39d4946a-74a0-412b-8dfb-423b23371da5"
-					(reference "R7")
-					(unit 1)
-				)

Commit message: Signed-off-by: SMAUG\Pete <pwbrophy@gmail.com>
Parts:
- C17, C2, C26, C27, C28, C29, C30, C31: JLCPCB Part # (none) -> C1779
- D9: footprint LED_SMD:LED_Kingbright_APA1606_1.6x0.6mm_Horizontal -> Diode_SMD:D_0603_1608Metric; JLCPCB Part # C965860 -> C2286; MANUFACTURER XINGLIGHT -> Hubei; Manufacturer_Part_Number XL-1606SURC -> KT-0603R
- J1, J2, J3, J4, J5, J7: now not fitted; now left out of the parts list
- R1, R12, R2, R20, R21, R22, R5, R6: JLCPCB Part # (none) -> C23182
- R10, R11, R13, R14, R18, R19, R8, R9: footprint Resistor_SMD:R_01005_0402Metric -> Resistor_SMD:R_0603_1608Metric; JLCPCB Part # C25744 -> C25804; Manufacturer_Part_Number 0402WGF1002TCE -> 0603WAF1002T5E
Connections:
- net +3V3_HULL: no longer J1.3 (Pin_3), J1.4 (Pin_4), J7.1 (Pin_1), J7.2 (Pin_2), U8.22 (SCL), U8.23 (SDA)
- net GND: now also C29.1, C31.1
- new net SCL: J1.4 (Pin_4), J7.1 (Pin_1), U8.22 (SCL)
- new net SDA: J1.3 (Pin_3), J7.2 (Pin_2), U8.23 (SDA)
- no-connect marks 7 -> 8

Commit message: Signed-off-by: SMAUG\Pete <pwbrophy@gmail.com>
Parts:
- TP3, TP4, TP5, TP6, TP7, TP8: now left out of the parts list
Changed lines of the file:
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@@
 		(unit 1)
 		(exclude_from_sim no)
-		(in_bom yes)
-		(on_board no)
+		(in_bom no)
+		(on_board yes)
 		(dnp yes)
 		(fields_autoplaced yes)
@@
 		(unit 1)
 		(exclude_from_sim no)
-		(in_bom yes)
-		(on_board no)
+		(in_bom no)
+		(on_board yes)
 		(dnp yes)
 		(fields_autoplaced yes)
@@
 		(unit 1)
 		(exclude_from_sim no)
-		(in_bom yes)
-		(on_board no)
+		(in_bom no)
+		(on_board yes)
 		(dnp yes)
 		(fields_autoplaced yes)
@@
 		(unit 1)
 		(exclude_from_sim no)
-		(in_bom yes)
-		(on_board no)
+		(in_bom no)
+		(on_board yes)
 		(dnp yes)
 		(property "Reference" "TP6"
@@
 		(unit 1)
 		(exclude_from_sim no)
-		(in_bom yes)
-		(on_board no)
+		(in_bom no)
+		(on_board yes)
 		(dnp yes)
 		(fields_autoplaced yes)
@@
 		(unit 1)
 		(exclude_from_sim no)
-		(in_bom yes)
-		(on_board no)
+		(in_bom no)
+		(on_board yes)
 		(dnp yes)
 		(fields_autoplaced yes)

Commit message: Signed-off-by: SMAUG\Pete <pwbrophy@gmail.com>
Connections:
- net Left Motor Control 1: now also U3.9 (BIN1); no longer U3.16 (AIN1)
- net Left Motor Control 2: now also U3.10 (BIN2); no longer U3.15 (AIN2)
- net Turret Motor Control 1: now also U3.16 (AIN1); no longer U3.9 (BIN1)
- net Turret Motor Control 2: now also U3.15 (AIN2); no longer U3.10 (BIN2)
Changed lines of the file:
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@@
 	)
 	(junction
+		(at 254 58.42)
+		(diameter 0)
+		(color 0 0 0 0)
+	)
+	(junction
 		(at 346.71 127)
 		(diameter 0)
@@
 	(wire
 		(pts
-			(xy 186.69 241.3) (xy 193.04 241.3)
-		)
-		(stroke
-			(width 0)
-			(type default)
-		)
-	)
-	(wire
-		(pts
 			(xy 105.41 219.71) (xy 113.03 219.71)
 		)
@@
 	(wire
 		(pts
+			(xy 187.96 238.76) (xy 193.04 238.76)
+		)
+		(stroke
+			(width 0)
+			(type default)
+		)
+	)
+	(wire
+		(pts
 			(xy 54.61 77.47) (xy 58.42 77.47)
 		)
@@
 	(wire
 		(pts
+			(xy 254 58.42) (xy 260.35 58.42)
+		)
+		(stroke
+			(width 0)
+			(type default)
+		)
+	)
+	(wire
+		(pts
 			(xy 132.08 140.97) (xy 129.54 140.97)
 		)
@@
 	(wire
 		(pts
+			(xy 187.96 246.38) (xy 193.04 246.38)
+		)
+		(stroke
+			(width 0)
+			(type default)
+		)
+	)
+	(wire
+		(pts
 			(xy 363.22 63.5) (xy 346.71 63.5)
 		)
@@
 	(wire
 		(pts
-			(xy 186.69 238.76) (xy 193.04 238.76)
-		)
-		(stroke
-			(width 0)
-			(type default)
-		)
-	)
-	(wire
-		(pts
-			(xy 257.81 60.96) (xy 260.35 60.96)
+			(xy 254 60.96) (xy 260.35 60.96)
 		)
 		(stroke
@@
 	(wire
 		(pts
+			(xy 254 58.42) (xy 254 60.96)
+		)
+		(stroke
+			(width 0)
+			(type default)
+		)
+	)
+	(wire
+		(pts
 			(xy 208.28 254) (xy 208.28 257.81)
 		)
@@
 	(wire
 		(pts
-			(xy 248.92 58.42) (xy 260.35 58.42)
+			(xy 248.92 58.42) (xy 254 58.42)
+		)
+		(stroke
+			(width 0)
+			(type default)
+		)
+	)
+	(wire
+		(pts
+			(xy 187.96 243.84) (xy 193.04 243.84)
 		)
 		(stroke
@@
 	(wire
 		(pts
+			(xy 187.96 241.3) (xy 193.04 241.3)
+		)
+		(stroke
+			(width 0)
+			(type default)
+		)
+	)
+	(wire
+		(pts
 			(xy 288.29 60.96) (xy 300.99 60.96)
 		)
@@
 	(wire
 		(pts
-			(xy 186.69 246.38) (xy 193.04 246.38)
-		)
-		(stroke
-			(width 0)
-			(type default)
-		)
-	)
-	(wire
-		(pts
 			(xy 147.32 69.85) (xy 147.32 74.93)
 		)
@@
 	(wire
 		(pts
-			(xy 186.69 243.84) (xy 193.04 243.84)
-		)
-		(stroke
-			(width 0)
-			(type default)
-		)
-	)
-	(wire
-		(pts
 			(xy 232.41 55.88) (xy 240.03 55.88)
 		)
@@
 	)
 	(label "Left Motor Control 2"
-		(at 186.69 241.3 180)
+		(at 187.96 246.38 180)
 		(effects
 			(font
@@
 	)
 	(label "Left Motor Control 1"
-		(at 186.69 238.76 180)
+		(at 187.96 243.84 180)
 		(effects
 			(font
@@
 	)
 	(label "Turret Motor Control 2"
-		(at 186.69 246.38 180)
+		(at 187.96 241.3 180)
 		(effects
 			(font
@@
 	)
 	(label "Turret Motor Control 1"
-		(at 186.69 243.84 180)
+		(at 187.96 238.76 180)
 		(effects
 			(font
@@
 					(unit 1)
 				)
-			)
-		)
-	)
-	(symbol
-		(lib_id "power:+BATT")
-		(at 257.81 60.96 90)
-		(unit 1)
-		(exclude_from_sim no)
-		(in_bom yes)
-		(on_board yes)
-		(dnp no)
-		(property "Reference" "#PWR031"
-			(at 261.62 60.96 0)
-			(effects
-				(font
-					(size 1.27 1.27)
-				)
-				(hide yes)
-			)
-		)
-		(property "Value" "+BATT"
-			(at 256.794 65.024 0)
-			(effects
-				(font
-					(size 1.27 1.27)
-				)
-			)
-		)
-		(property "Footprint" ""
-			(at 257.81 60.96 0)
-			(effects
-				(font
-					(size 1.27 1.27)
-				)
-				(hide yes)
-			)
-		)
-		(property "Datasheet" ""
-			(at 257.81 60.96 0)
-			(effects
-				(font
-					(size 1.27 1.27)
-				)
-				(hide yes)
-			)
-		)
-		(property "Description" "Power symbol creates a global label with name \"+BATT\""
-			(at 257.81 60.96 0)
-			(effects
-				(font
-					(size 1.27 1.27)
-				)
-				(hide yes)
-			)
-		)
-		(pin "1"
-		)
-		(instances
-			(project "TankHull"
-				(path "/39d4946a-74a0-412b-8dfb-423b23371da5"
-					(reference "#PWR031")
-					(unit 1)
-				)

Commit message: Signed-off-by: SMAUG\Pete <pwbrophy@gmail.com>
Parts:
- added D4: LED, LED_SMD:LED_0805_2012Metric, symbol Device:LED
- added R23, R24, R25, R26, R27, R3, R7: 10kΩ, Resistor_SMD:R_0603_1608Metric, symbol Device:R
- added R28: 220, Resistor_SMD:R_0603_1608Metric, symbol Device:R
- J1, J2, J3, J4, J5: now fitted; now in the parts list
- U10, U11, U12, U4, U5, U6, U7, U9: JLCPCB C499566 -> (none)
Connections:
- net GND: now also U2.15 (AIN2), U2.16 (AIN1), D4.1 (K), R23.1, R24.2, R25.2, R26.2, R27.2, R3.2, R7.2
- net Left Motor Control 1: now also U8.15 (IO1_2), R23.2; no longer U8.13 (IO1_0)
- net Left Motor Control 2: now also U8.16 (IO1_3), R7.1; no longer U8.14 (IO1_1)
- net Motors Sleep: now also R27.1
- net Right Motor Control 1: now also R25.1
- net Right Motor Control 2: now also R26.1
- net Turret Motor Control 1: now also U8.13 (IO1_0), R3.1; no longer U8.15 (IO1_2)
- net Turret Motor Control 2: now also U8.14 (IO1_1), R24.1; no longer U8.16 (IO1_3)
- net at U8.20 (IO1_7): now also R28.2
- new net: D4.2 (A), R28.1
- no-connect marks 8 -> 5
Other:
- note added: "GREEN GPIO"
- moved on the sheet: C11, C12, C6, C8, TP3, TP4, TP5, TP6, TP7, U3

Commit message: Signed-off-by: SMAUG\Pete <pwbrophy@gmail.com>
Parts:
- removed Q1: Q_PMOS, Package_TO_SOT_SMD:SOT-23-3, symbol Device:Q_PMOS
- added Q2: AO3401A, EasyEDA2Kicad:SOT-23_L2.9-W1.3-P1.90-LS2.4-BR, symbol EasyEDA2Kicad:AO3401A
- added TP1: TestPoint, TestPoint:TestPoint_Pad_D1.0mm, symbol Connector:TestPoint
- J1: footprint Connector_JST:JST_XH_B4B-XH-A_1x04_P2.50mm_Vertical -> Connector_JST:JST_PH_B5B-PH-K_1x05_P2.00mm_Vertical; symbol Connector_Generic:Conn_02x02_Odd_Even -> Connector:Conn_01x05_Socket; JLCPCB Part # C2908602 -> C157993
Connections:
- net +BATT: now also Q2.2 (S)
- net SCL: now also J1.5 (Pin_5); no longer J1.4 (Pin_4)
- net SDA: now also J1.4 (Pin_4); no longer J1.3 (Pin_3)
- net VBAT_RAW: now also Q2.3 (D)
- net INT: now reaches U8.1 (~{INT})
- net INT: now also J1.3 (Pin_3), TP1.1
- net at R4.1: now also Q2.1 (G)
- no-connect marks 5 -> 4

Commit message: V0.2 Files sent to JLC PCB on 15/03/2026
Parts:
- J1: Manufacturer_Part_Number XH-4A -> (none)
- Q2: JLCPCB Part # (none) -> C15127; LCSC Part C15127 -> (none)
- R28: value 220 -> 220Ω
Changed lines of the file:
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@@
 	(wire
 		(pts
+			(xy 64.77 227.33) (xy 69.85 227.33)
+		)
+		(stroke
+			(width 0)
+			(type default)
+		)
+	)
+	(wire
+		(pts
 			(xy 54.61 74.93) (xy 58.42 74.93)
 		)
@@
 	(wire
 		(pts
-			(xy 234.95 217.17) (xy 234.95 218.44)
+			(xy 346.71 107.95) (xy 346.71 109.22)
 		)
 		(stroke
@@
 	(wire
 		(pts
-			(xy 346.71 107.95) (xy 346.71 109.22)
+			(xy 55.88 247.65) (xy 58.42 247.65)
 		)
 		(stroke
@@
 	(wire
 		(pts
-			(xy 55.88 247.65) (xy 58.42 247.65)
+			(xy 323.85 91.44) (xy 323.85 109.22)
 		)
 		(stroke
@@
 	(wire
 		(pts
-			(xy 323.85 91.44) (xy 323.85 109.22)
+			(xy 67.31 232.41) (xy 67.31 234.95)
 		)
 		(stroke
@@
 	(wire
 		(pts
-			(xy 67.31 232.41) (xy 67.31 234.95)
+			(xy 339.09 63.5) (xy 346.71 63.5)
 		)
 		(stroke
@@
 	(wire
 		(pts
-			(xy 339.09 63.5) (xy 346.71 63.5)
+			(xy 346.71 160.02) (xy 346.71 162.56)
 		)
 		(stroke
@@
 	(wire
 		(pts
-			(xy 346.71 160.02) (xy 346.71 162.56)
+			(xy 176.53 143.51) (xy 176.53 148.59)
 		)
 		(stroke
@@
 	(wire
 		(pts
-			(xy 176.53 143.51) (xy 176.53 148.59)
+			(xy 234.95 217.17) (xy 234.95 218.44)
 		)
 		(stroke
@@
 	)
 	(label "Motors Sleep"
-		(at 69.85 227.33 180)
+		(at 64.77 227.33 180)
 		(effects
 			(font
@@
 			)
 		)
-		(property "Value" "220"
+		(property "Value" "220Ω"
 			(at 112.014 166.37 90)
 			(effects
@@
 			)
 		)
-		(property "LCSC Part" "C15127"
+		(property "LCSC Part" ""
 			(at 165.1 54.61 0)
 			(effects
@@
 			)
 		)
+		(property "JLCPCB Part #" "C15127"
+			(at 147.32 54.61 90)
+			(effects
+				(font
+					(size 1.27 1.27)
+				)
+				(hide yes)
+			)
+		)
 		(pin "3"
 		)
@@
 			)
 		)
-		(property "Manufacturer_Part_Number" "XH-4A"
+		(property "Manufacturer_Part_Number" ""
 			(at 74.422 40.894 0)
 			(effects
